Commit message: feat: finishing up the GA

File: evolving_creatures/URDF/0.urdf (robot description, URDF)
Before this commit: robot ted, 9 links, 8 joints
Links:
- link 0: mass 0.2412296096159241 -> 0.5301131038898502; geometry collision cylinder length=0.6708473124047619 radius=0.5355623986449429; visual cylinder length=0.6708473124047619 radius=0.5355623986449429
- link 11: mass 0.03348456968220448 -> 0.6608165995406313; geometry collision cylinder length=0.750495612183022 radius=0.7761980235104629; visual cylinder length=0.750495612183022 radius=0.7761980235104629
- link 15: mass 0.03348456968220448 -> 0.6608165995406313; geometry collision cylinder length=0.750495612183022 radius=0.7761980235104629; visual cylinder length=0.750495612183022 radius=0.7761980235104629
- link 22: mass 0.3347560652499726 -> 0.36466399389028514; geometry collision cylinder length=0.5363185494668233 radius=0.2766123611849439; visual cylinder length=0.5363185494668233 radius=0.2766123611849439
- link 23: mass 0.3347560652499726 -> 0.36466399389028514; geometry collision cylinder length=0.5363185494668233 radius=0.2766123611849439; visual cylinder length=0.5363185494668233 radius=0.2766123611849439
- link 24: mass 0.3347560652499726 -> 0.36466399389028514; geometry collision cylinder length=0.5363185494668233 radius=0.2766123611849439; visual cylinder length=0.5363185494668233 radius=0.2766123611849439
- link 26: mass 0.3347560652499726 -> 0.36466399389028514; geometry collision cylinder length=0.5363185494668233 radius=0.2766123611849439; visual cylinder length=0.5363185494668233 radius=0.2766123611849439
- link 27: mass 0.3347560652499726 -> 0.36466399389028514; geometry collision cylinder length=0.5363185494668233 radius=0.2766123611849439; visual cylinder length=0.5363185494668233 radius=0.2766123611849439
- link 28: mass 0.3347560652499726 -> 0.36466399389028514; geometry collision cylinder length=0.5363185494668233 radius=0.2766123611849439; visual cylinder length=0.5363185494668233 radius=0.2766123611849439
Joints:
- joint 0_to_11: origin xyz=0.5826968548142001 0.7319186353717901 0.2558917238483778 rpy=7.052425458248692 2.6296361898905904 4.506113772165355 -> xyz=0.904066690124414 0.49412361786727677 0.5722745687416606 rpy=11.584333380566894 1.932982834810668 4.437734220967872
- joint 0_to_15: origin xyz=0.5826968548142001 0.7319186353717901 0.2558917238483778 rpy=10.578638187373038 2.6296361898905904 4.506113772165355 -> xyz=0.904066690124414 0.49412361786727677 0.5722745687416606 rpy=17.37650007085034 1.932982834810668 4.437734220967872
- joint 11_to_22: origin xyz=0.7518519160738443 0.05442155615922484 0.04235412016236306 rpy=3.6117890591241237 1.6373332929494908 4.089191677937729 -> xyz=0.6319107371297262 0.6266655193750771 0.9152500838659247 rpy=10.565530740733406 2.483966454281209 2.496973003856025; type fixed -> revolute
- joint 11_to_23: origin xyz=0.7518519160738443 0.05442155615922484 0.04235412016236306 rpy=5.417683588686185 1.6373332929494908 4.089191677937729 -> xyz=0.6319107371297262 0.6266655193750771 0.9152500838659247 rpy=15.848296111100108 2.483966454281209 2.496973003856025; type fixed -> revolute
- joint 11_to_24: origin xyz=0.7518519160738443 0.05442155615922484 0.04235412016236306 rpy=7.2235781182482475 1.6373332929494908 4.089191677937729 -> xyz=0.6319107371297262 0.6266655193750771 0.9152500838659247 rpy=21.131061481466812 2.483966454281209 2.496973003856025; type fixed -> revolute
- joint 15_to_26: origin xyz=0.7518519160738443 0.05442155615922484 0.04235412016236306 rpy=3.6117890591241237 1.6373332929494908 4.089191677937729 -> xyz=0.6319107371297262 0.6266655193750771 0.9152500838659247 rpy=10.565530740733406 2.483966454281209 2.496973003856025; type fixed -> revolute
- joint 15_to_27: origin xyz=0.7518519160738443 0.05442155615922484 0.04235412016236306 rpy=5.417683588686185 1.6373332929494908 4.089191677937729 -> xyz=0.6319107371297262 0.6266655193750771 0.9152500838659247 rpy=15.848296111100108 2.483966454281209 2.496973003856025; type fixed -> revolute
- joint 15_to_28: origin xyz=0.7518519160738443 0.05442155615922484 0.04235412016236306 rpy=7.2235781182482475 1.6373332929494908 4.089191677937729 -> xyz=0.6319107371297262 0.6266655193750771 0.9152500838659247 rpy=21.131061481466812 2.483966454281209 2.496973003856025; type fixed -> revolute

File: evolving_creatures/URDF/1.urdf (robot description, URDF)
Before this commit: robot ted, 8 links, 7 joints
Links:
- removed link 12
- removed link 13
- removed link 25
- removed link 26
- removed link 27
- added link 22, mass 0.43293422327698383; collision cylinder length=0.5813812536232463 radius=0.9352171682302326; visual cylinder length=0.5813812536232463 radius=0.9352171682302326
- added link 23, mass 0.43293422327698383; collision cylinder length=0.5813812536232463 radius=0.9352171682302326; visual cylinder length=0.5813812536232463 radius=0.9352171682302326
- link 0: mass 0.6896900547839262 -> 0.23407871841241357; geometry collision cylinder length=0.9307606622335557 radius=0.612155293778461; visual cylinder length=0.9307606622335557 radius=0.612155293778461
- link 11: mass 0.30774240687557597 -> 0.4083755482210827; geometry collision cylinder length=0.45000327052615274 radius=0.875127749692599; visual cylinder length=0.45000327052615274 radius=0.875127749692599
- link 24: mass 0.9571704990539702 -> 0.43293422327698383; geometry collision cylinder length=0.5813812536232463 radius=0.9352171682302326; visual cylinder length=0.5813812536232463 radius=0.9352171682302326
Joints:
- removed joint 0_to_12
- removed joint 0_to_13
- removed joint 0_to_25
- removed joint 0_to_26
- removed joint 0_to_27
- added joint 0_to_22: type revolute, parent 0, child 22, origin xyz=0.33766691322269415 0.9268574764629836 0.5396408670947822 rpy=12.042250346720872 3.4761228631540915 4.603208052221171, axis 1 0 0, limit effort=1 velocity=1
- added joint 0_to_23: type revolute, parent 0, child 23, origin xyz=0.33766691322269415 0.9268574764629836 0.5396408670947822 rpy=16.05633379562783 3.4761228631540915 4.603208052221171, axis 1 0 0, limit effort=1 velocity=1
- joint 0_to_11: origin xyz=0.3155635908966845 0.3171267160949417 0.6503652802021906 rpy=5.765340755135096 0.15570354081100532 1.0225124473757625 -> xyz=0.5711361873981222 0.06355420971682557 0.8084972414942933 rpy=5.957113464629277 1.1621065363046357 5.3823881901385535
- joint 0_to_24: origin xyz=0.33491539078961763 0.17615761053248913 0.6511537444237424 rpy=12.176389204799422 1.7337999965568178 2.3563462578249164 -> xyz=0.33766691322269415 0.9268574764629836 0.5396408670947822 rpy=20.070417244534788 3.4761228631540915 4.603208052221171; type fixed -> revolute

File: evolving_creatures/URDF/10.urdf (robot description, URDF)
Before this commit: robot ted, 7 links, 6 joints
Links:
- removed link 12
- removed link 23
- removed link 25
- added link 13, mass 0.6747531513622993; collision cylinder length=0.35398580004262525 radius=0.5691309547641357; visual cylinder length=0.35398580004262525 radius=0.5691309547641357
- added link 15, mass 0.6747531513622993; collision cylinder length=0.35398580004262525 radius=0.5691309547641357; visual cylinder length=0.35398580004262525 radius=0.5691309547641357
- added link 22, mass 0.9561266460267444; collision cylinder length=0.3418419644097235 radius=0.20617160769999165; visual cylinder length=0.3418419644097235 radius=0.20617160769999165
- link 0: mass 0.587901268589428 -> 0.15993937193236452; geometry collision cylinder length=0.9873780067956286 radius=0.5561728234923146; visual cylinder length=0.9873780067956286 radius=0.5561728234923146
- link 11: mass 0.9148991792843637 -> 0.6747531513622993; geometry collision cylinder length=0.35398580004262525 radius=0.5691309547641357; visual cylinder length=0.35398580004262525 radius=0.5691309547641357
- link 24: mass 0.3823414554312763 -> 0.9561266460267444; geometry collision cylinder length=0.3418419644097235 radius=0.20617160769999165; visual cylinder length=0.3418419644097235 radius=0.20617160769999165
- link 26: mass 0.3823414554312763 -> 0.9561266460267444; geometry collision cylinder length=0.3418419644097235 radius=0.20617160769999165; visual cylinder length=0.3418419644097235 radius=0.20617160769999165
Joints:
- removed joint 0_to_12
- removed joint 0_to_23
- removed joint 0_to_24
- removed joint 0_to_25
- removed joint 0_to_26
- added joint 0_to_13: type fixed, parent 0, child 13, origin xyz=0.4101654414716812 0.5253715872288691 0.7782144858966138 rpy=12.2673763220681 5.490855656101748 0.4532833983370268, axis 1 0 0, limit effort=1 velocity=1
- added joint 0_to_15: type fixed, parent 0, child 15, origin xyz=0.4101654414716812 0.5253715872288691 0.7782144858966138 rpy=16.356501762757468 5.490855656101748 0.4532833983370268, axis 1 0 0, limit effort=1 velocity=1
- added joint 11_to_22: type fixed, parent 11, child 22, origin xyz=0.3169180888454084 0.27722928085200316 0.8708696303575072 rpy=0.8062508576953322 3.0069896662705813 0.7590698424267156, axis 1 0 0, limit effort=1 velocity=1
- added joint 13_to_24: type fixed, parent 13, child 24, origin xyz=0.3169180888454084 0.27722928085200316 0.8708696303575072 rpy=0.8062508576953322 3.0069896662705813 0.7590698424267156, axis 1 0 0, limit effort=1 velocity=1
- added joint 15_to_26: type fixed, parent 15, child 26, origin xyz=0.3169180888454084 0.27722928085200316 0.8708696303575072 rpy=0.8062508576953322 3.0069896662705813 0.7590698424267156, axis 1 0 0, limit effort=1 velocity=1
- joint 0_to_11: origin xyz=0.8432996132699462 0.3605896773412034 0.013661229417617937 rpy=12.456291431848484 1.5961664172502725 3.287303750934768 -> xyz=0.4101654414716812 0.5253715872288691 0.7782144858966138 rpy=8.178250881378734 5.490855656101748 0.4532833983370268

File: evolving_creatures/URDF/11.urdf (robot description, URDF)
Before this commit: robot ted, 6 links, 5 joints
Links:
- removed link 12
- removed link 13
- removed link 24
- removed link 25
- added link 22, mass 0.6075719086087558; collision cylinder length=0.33176793351724365 radius=0.7526736773168717; visual cylinder length=0.33176793351724365 radius=0.7526736773168717
- added link 23, mass 0.6075719086087558; collision cylinder length=0.33176793351724365 radius=0.7526736773168717; visual cylinder length=0.33176793351724365 radius=0.7526736773168717
- link 0: mass 0.4514554263737528 -> 0.7706508026362331; geometry collision cylinder length=0.3913382783131587 radius=0.32110501689661286; visual cylinder length=0.3913382783131587 radius=0.32110501689661286
- link 11: mass 0.07936963986223422 -> 0.8568659610022978; geometry collision cylinder length=0.8235975560681397 radius=0.653890846074599; visual cylinder length=0.8235975560681397 radius=0.653890846074599
Joints:
- removed joint 0_to_12
- removed joint 0_to_13
- removed joint 0_to_24
- removed joint 0_to_25
- added joint 0_to_22: type revolute, parent 0, child 22, origin xyz=0.4769501562542764 0.707279532225607 0.20012083186896712 rpy=3.506659171027442 0.6988158302917657 3.0689953436694184, axis 1 0 0, limit effort=1 velocity=1
- added joint 0_to_23: type revolute, parent 0, child 23, origin xyz=0.4769501562542764 0.707279532225607 0.20012083186896712 rpy=4.675545561369923 0.6988158302917657 3.0689953436694184, axis 1 0 0, limit effort=1 velocity=1
- joint 0_to_11: origin xyz=0.6497501915653128 0.08149909432804503 0.0650383780737015 rpy=0.19184290132456644 0.413924530656532 0.5492033803701684 -> xyz=0.7741562164640292 0.48507474038404597 0.577923795406728 rpy=4.586103516151838 4.549414251395375 0.5346246509624677

File: evolving_creatures/URDF/2.urdf (robot description, URDF)
Before this commit: robot ted, 9 links, 8 joints
Links:
- removed link 15
- removed link 22
- removed link 23
- removed link 24
- added link 12, mass 0.02649475875294538; collision cylinder length=0.042797832434671834 radius=0.9870472196025623; visual cylinder length=0.042797832434671834 radius=0.9870472196025623
- added link 13, mass 0.02649475875294538; collision cylinder length=0.042797832434671834 radius=0.9870472196025623; visual cylinder length=0.042797832434671834 radius=0.9870472196025623
- added link 14, mass 0.02649475875294538; collision cylinder length=0.042797832434671834 radius=0.9870472196025623; visual cylinder length=0.042797832434671834 radius=0.9870472196025623
- added link 25, mass 0.7997861727955152; collision cylinder length=0.0033241599462673355 radius=0.43409758858946834; visual cylinder length=0.0033241599462673355 radius=0.43409758858946834
- link 0: mass 0.017873426309739315 -> 0.46066775353622313; geometry collision cylinder length=0.28398240251131923 radius=0.7390878413404952; visual cylinder length=0.28398240251131923 radius=0.7390878413404952
- link 11: mass 0.28034976706710757 -> 0.02649475875294538; geometry collision cylinder length=0.042797832434671834 radius=0.9870472196025623; visual cylinder length=0.042797832434671834 radius=0.9870472196025623
- link 26: mass 0.24574800674891373 -> 0.7997861727955152; geometry collision cylinder length=0.0033241599462673355 radius=0.43409758858946834; visual cylinder length=0.0033241599462673355 radius=0.43409758858946834
- link 27: mass 0.24574800674891373 -> 0.7997861727955152; geometry collision cylinder length=0.0033241599462673355 radius=0.43409758858946834; visual cylinder length=0.0033241599462673355 radius=0.43409758858946834
- link 28: mass 0.24574800674891373 -> 0.7997861727955152; geometry collision cylinder length=0.0033241599462673355 radius=0.43409758858946834; visual cylinder length=0.0033241599462673355 radius=0.43409758858946834
Joints:
- removed joint 0_to_15
- removed joint 11_to_22
- removed joint 11_to_23
- removed joint 11_to_24
- removed joint 15_to_26
- removed joint 15_to_27
- removed joint 15_to_28
- added joint 0_to_12: type revolute, parent 0, child 12, origin xyz=0.07032620838734782 0.7247642311892147 0.3969425369952374 rpy=5.229940534973439 3.1845115729762425 1.870276071862189, axis 1 0 0, limit effort=1 velocity=1
- added joint 0_to_13: type revolute, parent 0, child 13, origin xyz=0.07032620838734782 0.7247642311892147 0.3969425369952374 rpy=6.9732540466312525 3.1845115729762425 1.870276071862189, axis 1 0 0, limit effort=1 velocity=1
- added joint 0_to_14: type revolute, parent 0, child 14, origin xyz=0.07032620838734782 0.7247642311892147 0.3969425369952374 rpy=8.716567558289066 3.1845115729762425 1.870276071862189, axis 1 0 0, limit effort=1 velocity=1
- added joint 0_to_25: type fixed, parent 0, child 25, origin xyz=0.7423841743265314 0.5084425653916115 0.10457052155715774 rpy=16.01713458198456 6.1164764893119745 1.7471893296671286, axis 1 0 0, limit effort=1 velocity=1
- added joint 0_to_26: type fixed, parent 0, child 26, origin xyz=0.7423841743265314 0.5084425653916115 0.10457052155715774 rpy=18.686657012315322 6.1164764893119745 1.7471893296671286, axis 1 0 0, limit effort=1 velocity=1
- added joint 0_to_27: type fixed, parent 0, child 27, origin xyz=0.7423841743265314 0.5084425653916115 0.10457052155715774 rpy=21.35617944264608 6.1164764893119745 1.7471893296671286, axis 1 0 0, limit effort=1 velocity=1
- added joint 0_to_28: type fixed, parent 0, child 28, origin xyz=0.7423841743265314 0.5084425653916115 0.10457052155715774 rpy=24.02570187297684 6.1164764893119745 1.7471893296671286, axis 1 0 0, limit effort=1 velocity=1
- joint 0_to_11: origin xyz=0.8286945369337435 0.9243843885467775 0.1757245077634677 rpy=2.6172688368260846 3.6285646362503945 3.0206708215558318 -> xyz=0.07032620838734782 0.7247642311892147 0.3969425369952374 rpy=3.4866270233156262 3.1845115729762425 1.870276071862189

File: evolving_creatures/URDF/3.urdf (robot description, URDF)
Before this commit: robot ted, 7 links, 6 joints
Links:
- removed link 13
- removed link 15
- removed link 26
- added link 111, mass 0.42143478416734315; collision cylinder length=0.7799979584429653 radius=0.5986185121146569; visual cylinder length=0.7799979584429653 radius=0.5986185121146569
- added link 16, mass 0.42143478416734315; collision cylinder length=0.7799979584429653 radius=0.5986185121146569; visual cylinder length=0.7799979584429653 radius=0.5986185121146569
- added link 210, mass 0.8241987209167628; collision cylinder length=0.4545651918322573 radius=0.17144367791166415; visual cylinder length=0.4545651918322573 radius=0.17144367791166415
- added link 212, mass 0.8241987209167628; collision cylinder length=0.4545651918322573 radius=0.17144367791166415; visual cylinder length=0.4545651918322573 radius=0.17144367791166415
- added link 213, mass 0.8241987209167628; collision cylinder length=0.4545651918322573 radius=0.17144367791166415; visual cylinder length=0.4545651918322573 radius=0.17144367791166415
- added link 214, mass 0.8241987209167628; collision cylinder length=0.4545651918322573 radius=0.17144367791166415; visual cylinder length=0.4545651918322573 radius=0.17144367791166415
- added link 215, mass 0.8241987209167628; collision cylinder length=0.4545651918322573 radius=0.17144367791166415; visual cylinder length=0.4545651918322573 radius=0.17144367791166415
- added link 23, mass 0.8241987209167628; collision cylinder length=0.4545651918322573 radius=0.17144367791166415; visual cylinder length=0.4545651918322573 radius=0.17144367791166415
- added link 25, mass 0.8241987209167628; collision cylinder length=0.4545651918322573 radius=0.17144367791166415; visual cylinder length=0.4545651918322573 radius=0.17144367791166415
- added link 27, mass 0.8241987209167628; collision cylinder length=0.4545651918322573 radius=0.17144367791166415; visual cylinder length=0.4545651918322573 radius=0.17144367791166415
- added link 28, mass 0.8241987209167628; collision cylinder length=0.4545651918322573 radius=0.17144367791166415; visual cylinder length=0.4545651918322573 radius=0.17144367791166415
- added link 29, mass 0.8241987209167628; collision cylinder length=0.4545651918322573 radius=0.17144367791166415; visual cylinder length=0.4545651918322573 radius=0.17144367791166415
- link 0: mass 0.25557090861487364 -> 0.3504002401598274; geometry collision cylinder length=0.5962753807705925 radius=0.07679702040628522; visual cylinder length=0.5962753807705925 radius=0.07679702040628522
- link 11: mass 0.6127226568258675 -> 0.42143478416734315; geometry collision cylinder length=0.7799979584429653 radius=0.5986185121146569; visual cylinder length=0.7799979584429653 radius=0.5986185121146569
- link 22: mass 0.24348454094182403 -> 0.8241987209167628; geometry collision cylinder length=0.4545651918322573 radius=0.17144367791166415; visual cylinder length=0.4545651918322573 radius=0.17144367791166415
- link 24: mass 0.24348454094182403 -> 0.8241987209167628; geometry collision cylinder length=0.4545651918322573 radius=0.17144367791166415; visual cylinder length=0.4545651918322573 radius=0.17144367791166415
Joints:
- removed joint 0_to_13
- removed joint 0_to_15
- removed joint 13_to_24
- removed joint 15_to_26
- added joint 0_to_111: type revolute, parent 0, child 111, origin xyz=0.22053987618566806 0.11791418867024372 0.23443846621962516 rpy=17.80429309144295 1.9277776971095466 5.8172402069666, axis 1 0 0, limit effort=1 velocity=1
- added joint 0_to_16: type revolute, parent 0, child 16, origin xyz=0.22053987618566806 0.11791418867024372 0.23443846621962516 rpy=13.353219818582213 1.9277776971095466 5.8172402069666, axis 1 0 0, limit effort=1 velocity=1
- added joint 111_to_212: type revolute, parent 111, child 212, origin xyz=0.6128328431496726 0.8579141484636779 0.19547059967940184 rpy=0.4149937271165128 1.5386317593199765 1.9275806566083498, axis 1 0 0, limit effort=1 velocity=1
- added joint 111_to_213: type revolute, parent 111, child 213, origin xyz=0.6128328431496726 0.8579141484636779 0.19547059967940184 rpy=0.6224905906747692 1.5386317593199765 1.9275806566083498, axis 1 0 0, limit effort=1 velocity=1
- added joint 111_to_214: type revolute, parent 111, child 214, origin xyz=0.6128328431496726 0.8579141484636779 0.19547059967940184 rpy=0.8299874542330256 1.5386317593199765 1.9275806566083498, axis 1 0 0, limit effort=1 velocity=1
- added joint 111_to_215: type revolute, parent 111, child 215, origin xyz=0.6128328431496726 0.8579141484636779 0.19547059967940184 rpy=1.037484317791282 1.5386317593199765 1.9275806566083498, axis 1 0 0, limit effort=1 velocity=1
- added joint 11_to_23: type revolute, parent 11, child 23, origin xyz=0.6128328431496726 0.8579141484636779 0.19547059967940184 rpy=0.6224905906747692 1.5386317593199765 1.9275806566083498, axis 1 0 0, limit effort=1 velocity=1
- added joint 11_to_24: type revolute, parent 11, child 24, origin xyz=0.6128328431496726 0.8579141484636779 0.19547059967940184 rpy=0.8299874542330256 1.5386317593199765 1.9275806566083498, axis 1 0 0, limit effort=1 velocity=1
- added joint 11_to_25: type revolute, parent 11, child 25, origin xyz=0.6128328431496726 0.8579141484636779 0.19547059967940184 rpy=1.037484317791282 1.5386317593199765 1.9275806566083498, axis 1 0 0, limit effort=1 velocity=1
- added joint 16_to_210: type revolute, parent 16, child 210, origin xyz=0.6128328431496726 0.8579141484636779 0.19547059967940184 rpy=1.037484317791282 1.5386317593199765 1.9275806566083498, axis 1 0 0, limit effort=1 velocity=1
- added joint 16_to_27: type revolute, parent 16, child 27, origin xyz=0.6128328431496726 0.8579141484636779 0.19547059967940184 rpy=0.4149937271165128 1.5386317593199765 1.9275806566083498, axis 1 0 0, limit effort=1 velocity=1
- added joint 16_to_28: type revolute, parent 16, child 28, origin xyz=0.6128328431496726 0.8579141484636779 0.19547059967940184 rpy=0.6224905906747692 1.5386317593199765 1.9275806566083498, axis 1 0 0, limit effort=1 velocity=1
- added joint 16_to_29: type revolute, parent 16, child 29, origin xyz=0.6128328431496726 0.8579141484636779 0.19547059967940184 rpy=0.8299874542330256 1.5386317593199765 1.9275806566083498, axis 1 0 0, limit effort=1 velocity=1
- joint 0_to_11: origin xyz=0.906111785756376 0.6088507627519042 0.8074769347017581 rpy=10.482826076826889 1.1928635817862638 3.7910199246240417 -> xyz=0.22053987618566806 0.11791418867024372 0.23443846621962516 rpy=8.902146545721475 1.9277776971095466 5.8172402069666
- joint 11_to_22: origin xyz=0.42934882003675234 0.5938646043363082 0.40037446801187415 rpy=5.0912508561899035 4.482540211693693 2.5212869038653714 -> xyz=0.6128328431496726 0.8579141484636779 0.19547059967940184 rpy=0.4149937271165128 1.5386317593199765 1.9275806566083498; type fixed -> revolute
