Commit message: feat: finishing up the GA

File: evolving_creatures/URDF/4.urdf (robot description, URDF)
Before this commit: robot ted, 5 links, 4 joints
Links:
- removed link 13
- added link 23, mass 0.06380921589664346; collision cylinder length=0.8652803744542434 radius=0.4655394501434208; visual cylinder length=0.8652803744542434 radius=0.4655394501434208
- added link 25, mass 0.06380921589664346; collision cylinder length=0.8652803744542434 radius=0.4655394501434208; visual cylinder length=0.8652803744542434 radius=0.4655394501434208
- link 0: mass 0.20040804230037224 -> 0.14180934674196166; geometry collision cylinder length=0.5658728723357201 radius=0.1955584258948394; visual cylinder length=0.5658728723357201 radius=0.1955584258948394
- link 11: mass 0.4101187942103659 -> 0.534972790434655; geometry collision cylinder length=0.3783565146551313 radius=0.3085258477925369; visual cylinder length=0.3783565146551313 radius=0.3085258477925369
- link 22: mass 0.8666044093986242 -> 0.06380921589664346; geometry collision cylinder length=0.8652803744542434 radius=0.4655394501434208; visual cylinder length=0.8652803744542434 radius=0.4655394501434208
- link 24: mass 0.8666044093986242 -> 0.06380921589664346; geometry collision cylinder length=0.8652803744542434 radius=0.4655394501434208; visual cylinder length=0.8652803744542434 radius=0.4655394501434208
Joints:
- removed joint 0_to_13
- removed joint 11_to_22
- removed joint 13_to_24
- added joint 0_to_22: type revolute, parent 0, child 22, origin xyz=0.41708751624837337 0.2729424412425584 0.37653101111524145 rpy=9.559121861997413 4.654915443752919 5.492102698234696, axis 1 0 0, limit effort=1 velocity=1
- added joint 0_to_23: type revolute, parent 0, child 23, origin xyz=0.41708751624837337 0.2729424412425584 0.37653101111524145 rpy=12.74549581599655 4.654915443752919 5.492102698234696, axis 1 0 0, limit effort=1 velocity=1
- added joint 0_to_24: type revolute, parent 0, child 24, origin xyz=0.41708751624837337 0.2729424412425584 0.37653101111524145 rpy=15.931869769995687 4.654915443752919 5.492102698234696, axis 1 0 0, limit effort=1 velocity=1
- added joint 0_to_25: type revolute, parent 0, child 25, origin xyz=0.41708751624837337 0.2729424412425584 0.37653101111524145 rpy=19.118243723994826 4.654915443752919 5.492102698234696, axis 1 0 0, limit effort=1 velocity=1
- joint 0_to_11: origin xyz=0.09372381634914051 0.06267976152252164 0.9551972440053589 rpy=9.124570646585411 3.9609163029744696 1.757882737548315 -> xyz=0.3624374404986638 0.6453773044998639 0.9820768054447729 rpy=12.41940327732792 0.7824432055021442 1.854183783044236; type revolute -> fixed

File: evolving_creatures/URDF/5.urdf (robot description, URDF)
Before this commit: robot ted, 5 links, 4 joints
Links:
- link 0: mass 0.45939679572431935 -> 0.5915219888699443; geometry collision cylinder length=0.9397554022476087 radius=0.5474820718989449; visual cylinder length=0.9397554022476087 radius=0.5474820718989449
- link 11: mass 0.36807050749833503 -> 0.5587351277461894; geometry collision cylinder length=0.26615686352681733 radius=0.1592615699535338; visual cylinder length=0.26615686352681733 radius=0.1592615699535338
- link 22: mass 0.03573135066767852 -> 0.5927891381067416; geometry collision cylinder length=0.2048360851532155 radius=0.8249099208052233; visual cylinder length=0.2048360851532155 radius=0.8249099208052233
- link 23: mass 0.03573135066767852 -> 0.5927891381067416; geometry collision cylinder length=0.2048360851532155 radius=0.8249099208052233; visual cylinder length=0.2048360851532155 radius=0.8249099208052233
- link 24: mass 0.03573135066767852 -> 0.5927891381067416; geometry collision cylinder length=0.2048360851532155 radius=0.8249099208052233; visual cylinder length=0.2048360851532155 radius=0.8249099208052233
Joints:
- removed joint 0_to_22
- removed joint 0_to_23
- removed joint 0_to_24
- added joint 11_to_22: type revolute, parent 11, child 22, origin xyz=0.67259057424336 0.10110383213590424 0.22809037119767928 rpy=1.2249424253303265 0.5355970113587686 2.813703567044261, axis 1 0 0, limit effort=1 velocity=1
- added joint 11_to_23: type revolute, parent 11, child 23, origin xyz=0.67259057424336 0.10110383213590424 0.22809037119767928 rpy=1.8374136379954897 0.5355970113587686 2.813703567044261, axis 1 0 0, limit effort=1 velocity=1
- added joint 11_to_24: type revolute, parent 11, child 24, origin xyz=0.67259057424336 0.10110383213590424 0.22809037119767928 rpy=2.449884850660653 0.5355970113587686 2.813703567044261, axis 1 0 0, limit effort=1 velocity=1
- joint 0_to_11: origin xyz=0.9104968082245044 0.8880739423737236 0.7791443113312373 rpy=1.2437489466869613 3.179511477570287 2.2897091328982997 -> xyz=0.9523668133272517 0.44254823454720327 0.25603083030857443 rpy=12.5325441779656 4.158678781984297 2.503122342430801; type revolute -> fixed

File: evolving_creatures/URDF/6.urdf (robot description, URDF)
Before this commit: robot ted, 3 links, 2 joints
Links:
- added link 14, mass 0.4771186923004319; collision cylinder length=0.8610294575730548 radius=0.3439519426486871; visual cylinder length=0.8610294575730548 radius=0.3439519426486871
- added link 17, mass 0.4771186923004319; collision cylinder length=0.8610294575730548 radius=0.3439519426486871; visual cylinder length=0.8610294575730548 radius=0.3439519426486871
- added link 23, mass 0.9911401011812869; collision cylinder length=0.6371326441123338 radius=0.25658454190482716; visual cylinder length=0.6371326441123338 radius=0.25658454190482716
- added link 25, mass 0.9911401011812869; collision cylinder length=0.6371326441123338 radius=0.25658454190482716; visual cylinder length=0.6371326441123338 radius=0.25658454190482716
- added link 26, mass 0.9911401011812869; collision cylinder length=0.6371326441123338 radius=0.25658454190482716; visual cylinder length=0.6371326441123338 radius=0.25658454190482716
- added link 28, mass 0.9911401011812869; collision cylinder length=0.6371326441123338 radius=0.25658454190482716; visual cylinder length=0.6371326441123338 radius=0.25658454190482716
- added link 29, mass 0.9911401011812869; collision cylinder length=0.6371326441123338 radius=0.25658454190482716; visual cylinder length=0.6371326441123338 radius=0.25658454190482716
- link 0: mass 0.26930780698329493 -> 0.9416563593579919; geometry collision cylinder length=0.27337669487151584 radius=0.5634259829770796; visual cylinder length=0.27337669487151584 radius=0.5634259829770796
- link 11: mass 0.42071888053124684 -> 0.4771186923004319; geometry collision cylinder length=0.8610294575730548 radius=0.3439519426486871; visual cylinder length=0.8610294575730548 radius=0.3439519426486871
- link 22: mass 0.5775649229263259 -> 0.9911401011812869; geometry collision cylinder length=0.6371326441123338 radius=0.25658454190482716; visual cylinder length=0.6371326441123338 radius=0.25658454190482716
Joints:
- added joint 0_to_14: type fixed, parent 0, child 14, origin xyz=0.35982983696756854 0.4948210628693771 0.17870137160170452 rpy=5.819441842083402 2.4397698640646737 2.7651980699006025, axis 1 0 0, limit effort=1 velocity=1
- added joint 0_to_17: type fixed, parent 0, child 17, origin xyz=0.35982983696756854 0.4948210628693771 0.17870137160170452 rpy=7.759255789444537 2.4397698640646737 2.7651980699006025, axis 1 0 0, limit effort=1 velocity=1
- added joint 11_to_23: type revolute, parent 11, child 23, origin xyz=0.4957513689821834 0.4331426638181324 0.6581422151439972 rpy=16.43156557353417 4.713583049832389 0.8825021323515916, axis 1 0 0, limit effort=1 velocity=1
- added joint 14_to_25: type revolute, parent 14, child 25, origin xyz=0.4957513689821834 0.4331426638181324 0.6581422151439972 rpy=10.95437704902278 4.713583049832389 0.8825021323515916, axis 1 0 0, limit effort=1 velocity=1
- added joint 14_to_26: type revolute, parent 14, child 26, origin xyz=0.4957513689821834 0.4331426638181324 0.6581422151439972 rpy=16.43156557353417 4.713583049832389 0.8825021323515916, axis 1 0 0, limit effort=1 velocity=1
- added joint 17_to_28: type revolute, parent 17, child 28, origin xyz=0.4957513689821834 0.4331426638181324 0.6581422151439972 rpy=10.95437704902278 4.713583049832389 0.8825021323515916, axis 1 0 0, limit effort=1 velocity=1
- added joint 17_to_29: type revolute, parent 17, child 29, origin xyz=0.4957513689821834 0.4331426638181324 0.6581422151439972 rpy=16.43156557353417 4.713583049832389 0.8825021323515916, axis 1 0 0, limit effort=1 velocity=1
- joint 0_to_11: origin xyz=0.6131601569090264 0.635322113696598 0.6758104740682828 rpy=9.952891875863138 3.4420643372295614 1.722549525986585 -> xyz=0.35982983696756854 0.4948210628693771 0.17870137160170452 rpy=3.8796278947222684 2.4397698640646737 2.7651980699006025; type revolute -> fixed
- joint 11_to_22: origin xyz=0.7301470040076475 0.439146727827623 0.5607710244391353 rpy=7.576945201360048 2.881128569817142 1.7876134810044841 -> xyz=0.4957513689821834 0.4331426638181324 0.6581422151439972 rpy=10.95437704902278 4.713583049832389 0.8825021323515916

File: evolving_creatures/URDF/7.urdf (robot description, URDF)
Before this commit: robot ted, 7 links, 6 joints
Links:
- link 0: mass 0.3935946548676942 -> 0.05787979911680308; geometry collision cylinder length=0.24444525882237378 radius=0.5903946241826806; visual cylinder length=0.24444525882237378 radius=0.5903946241826806
- link 11: mass 0.9014012552777548 -> 0.4053506420887715; geometry collision cylinder length=0.20971072817688596 radius=0.3545763251454792; visual cylinder length=0.20971072817688596 radius=0.3545763251454792
- link 12: mass 0.9014012552777548 -> 0.4053506420887715; geometry collision cylinder length=0.20971072817688596 radius=0.3545763251454792; visual cylinder length=0.20971072817688596 radius=0.3545763251454792
- link 13: mass 0.9014012552777548 -> 0.4053506420887715; geometry collision cylinder length=0.20971072817688596 radius=0.3545763251454792; visual cylinder length=0.20971072817688596 radius=0.3545763251454792
- link 14: mass 0.9014012552777548 -> 0.4053506420887715; geometry collision cylinder length=0.20971072817688596 radius=0.3545763251454792; visual cylinder length=0.20971072817688596 radius=0.3545763251454792
- link 25: mass 0.8947832574563347 -> 0.5560371678881377; geometry collision cylinder length=0.45530324497069463 radius=0.1728710910442851; visual cylinder length=0.45530324497069463 radius=0.1728710910442851
- link 26: mass 0.8947832574563347 -> 0.5560371678881377; geometry collision cylinder length=0.45530324497069463 radius=0.1728710910442851; visual cylinder length=0.45530324497069463 radius=0.1728710910442851
Joints:
- joint 0_to_11: origin xyz=0.770172108080939 0.8462387172466617 0.9739261721034488 rpy=0.5863936291898857 4.69806648274824 0.8247175925889169 -> xyz=0.24242234705389487 0.33828020878731035 0.2959242856990707 rpy=5.377656601893495 4.32067423514443 3.563202333276369
- joint 0_to_12: origin xyz=0.770172108080939 0.8462387172466617 0.9739261721034488 rpy=0.8795904437848285 4.69806648274824 0.8247175925889169 -> xyz=0.24242234705389487 0.33828020878731035 0.2959242856990707 rpy=8.066484902840243 4.32067423514443 3.563202333276369
- joint 0_to_13: origin xyz=0.770172108080939 0.8462387172466617 0.9739261721034488 rpy=1.1727872583797714 4.69806648274824 0.8247175925889169 -> xyz=0.24242234705389487 0.33828020878731035 0.2959242856990707 rpy=10.75531320378699 4.32067423514443 3.563202333276369
- joint 0_to_14: origin xyz=0.770172108080939 0.8462387172466617 0.9739261721034488 rpy=1.4659840729747142 4.69806648274824 0.8247175925889169 -> xyz=0.24242234705389487 0.33828020878731035 0.2959242856990707 rpy=13.444141504733738 4.32067423514443 3.563202333276369
- joint 0_to_25: origin xyz=0.16014508372725011 0.7462137259312588 0.662594928742491 rpy=27.36328307248862 0.3324729514883024 5.097917870326313 -> xyz=0.8326664985214015 0.1396020296978696 0.3874407679785091 rpy=20.585192229907925 0.36204938908470924 5.372293525679539
- joint 0_to_26: origin xyz=0.16014508372725011 0.7462137259312588 0.662594928742491 rpy=31.923830251236723 0.3324729514883024 5.097917870326313 -> xyz=0.8326664985214015 0.1396020296978696 0.3874407679785091 rpy=24.016057601559243 0.36204938908470924 5.372293525679539

File: evolving_creatures/URDF/8.urdf (robot description, URDF)
Before this commit: robot ted, 17 links, 16 joints
Links:
- removed link 113
- removed link 15
- removed link 19
- removed link 210
- removed link 211
- removed link 212
- removed link 214
- removed link 215
- removed link 216
- removed link 24
- removed link 26
- removed link 27
- removed link 28
- link 0: mass 0.9048998964019388 -> 0.918851376352353; geometry collision cylinder length=0.6429270423449143 radius=0.9710204988893348; visual cylinder length=0.6429270423449143 radius=0.9710204988893348
- link 11: mass 0.4026650594801602 -> 0.5869899911583579; geometry collision cylinder length=0.18528122135910685 radius=0.08685378833162605; visual cylinder length=0.18528122135910685 radius=0.08685378833162605
- link 22: mass 0.4419140350426659 -> 0.17690250276246489; geometry collision cylinder length=0.6225128736817918 radius=0.2840788856534705; visual cylinder length=0.6225128736817918 radius=0.2840788856534705
- link 23: mass 0.4419140350426659 -> 0.17690250276246489; geometry collision cylinder length=0.6225128736817918 radius=0.2840788856534705; visual cylinder length=0.6225128736817918 radius=0.2840788856534705
Joints:
- removed joint 0_to_113
- removed joint 0_to_15
- removed joint 0_to_19
- removed joint 113_to_214
- removed joint 113_to_215
- removed joint 113_to_216
- removed joint 11_to_24
- removed joint 15_to_26
- removed joint 15_to_27
- removed joint 15_to_28
- removed joint 19_to_210
- removed joint 19_to_211
- removed joint 19_to_212
- joint 0_to_11: origin xyz=0.3947269811845817 0.5387657059059537 0.5119870247011911 rpy=1.2623274237396314 0.3336954673981916 0.07359562693552224 -> xyz=0.31356293640167177 0.7714657555208229 0.746370997194334 rpy=12.367558002888956 0.367235277655106 4.608598057269663
- joint 11_to_22: origin xyz=0.06953930004845932 0.9894687917997325 0.3042457931526853 rpy=10.412136958944581 5.375376994199804 2.4057046627266865 -> xyz=0.650671638412766 0.939345301046582 0.7191100530265305 rpy=1.676996027096198 5.843553322684614 1.5541850768214387
- joint 11_to_23: origin xyz=0.06953930004845932 0.9894687917997325 0.3042457931526853 rpy=15.618205438416872 5.375376994199804 2.4057046627266865 -> xyz=0.650671638412766 0.939345301046582 0.7191100530265305 rpy=2.515494040644297 5.843553322684614 1.5541850768214387

File: evolving_creatures/URDF/9.urdf (robot description, URDF)
Before this commit: robot ted, 9 links, 8 joints
Links:
- removed link 13
- removed link 15
- removed link 17
- removed link 22
- removed link 24
- removed link 26
- removed link 28
- added link 12, mass 0.1682654256186824; collision cylinder length=0.5298200372119601 radius=0.9061586023718584; visual cylinder length=0.5298200372119601 radius=0.9061586023718584
- added link 23, mass 0.5348341843777173; collision cylinder length=0.6917308004086973 radius=0.08620360313467035; visual cylinder length=0.6917308004086973 radius=0.08620360313467035
- link 0: mass 0.9709771733583835 -> 0.5727515049594439; geometry collision cylinder length=0.8572744288386839 radius=0.27774521493392745; visual cylinder length=0.8572744288386839 radius=0.27774521493392745
- link 11: mass 0.9929809530843084 -> 0.1682654256186824; geometry collision cylinder length=0.5298200372119601 radius=0.9061586023718584; visual cylinder length=0.5298200372119601 radius=0.9061586023718584
Joints:
- removed joint 0_to_13
- removed joint 0_to_15
- removed joint 0_to_17
- removed joint 11_to_22
- removed joint 13_to_24
- removed joint 15_to_26
- removed joint 17_to_28
- added joint 0_to_12: type revolute, parent 0, child 12, origin xyz=0.0854493099546173 0.5597876151517075 0.8133481299798041 rpy=14.891253683074707 2.9538544921693948 1.67510710532705, axis 1 0 0, limit effort=1 velocity=1
- added joint 0_to_23: type fixed, parent 0, child 23, origin xyz=0.8135121865456393 0.39925524710584415 0.6843857510679386 rpy=13.248666557600203 6.064974791973338 2.1507414822589466, axis 1 0 0, limit effort=1 velocity=1
- joint 0_to_11: origin xyz=0.33780074157543505 0.9833909730028172 0.5925596446223254 rpy=1.0568335645612275 1.7307946398975278 3.3740904726330516 -> xyz=0.0854493099546173 0.5597876151517075 0.8133481299798041 rpy=9.927502455383138 2.9538544921693948 1.67510710532705
