Commit message: finishing up

File: URDF/0.urdf (robot description, URDF)
Before this commit: robot ted, 9 links, 8 joints
Links:
- removed link 15
- removed link 22
- removed link 23
- removed link 24
- removed link 26
- removed link 27
- removed link 28
- added link 12, mass 0.11888556824783847; collision cylinder length=0.20148864524368926 radius=0.39336189641222474; visual cylinder length=0.20148864524368926 radius=0.39336189641222474
- added link 13, mass 0.11888556824783847; collision cylinder length=0.20148864524368926 radius=0.39336189641222474; visual cylinder length=0.20148864524368926 radius=0.39336189641222474
- link 0: mass 0.5301131038898502 -> -0.041928476734819975; geometry collision cylinder length=0.21275301331532537 radius=0.6738214328149634; visual cylinder length=0.21275301331532537 radius=0.6738214328149634
- link 11: mass 0.6608165995406313 -> 0.11888556824783847; geometry collision cylinder length=0.20148864524368926 radius=0.39336189641222474; visual cylinder length=0.20148864524368926 radius=0.39336189641222474
Joints:
- removed joint 0_to_15
- removed joint 11_to_22
- removed joint 11_to_23
- removed joint 11_to_24
- removed joint 15_to_26
- removed joint 15_to_27
- removed joint 15_to_28
- added joint 0_to_12: type revolute, parent 0, child 12, origin xyz=0.8406967620585992 0.17178042112934833 0.5677756171937046 rpy=1.5396977613382736 2.8809326456153213 2.0432824326917585, axis 1 0 0, limit effort=1 velocity=1
- added joint 0_to_13: type revolute, parent 0, child 13, origin xyz=0.8406967620585992 0.17178042112934833 0.5677756171937046 rpy=2.0529303484510315 2.8809326456153213 2.0432824326917585, axis 1 0 0, limit effort=1 velocity=1
- joint 0_to_11: origin xyz=0.904066690124414 0.49412361786727677 0.5722745687416606 rpy=11.584333380566894 1.932982834810668 4.437734220967872 -> xyz=0.8406967620585992 0.17178042112934833 0.5677756171937046 rpy=1.0264651742255158 2.8809326456153213 2.0432824326917585

File: URDF/1.urdf (robot description, URDF)
Before this commit: robot ted, 5 links, 4 joints
Links:
- removed link 22
- removed link 23
- removed link 24
- added link 12, mass 0.15762616033790156; collision cylinder length=0.3192604814356006 radius=0.4691899845299726; visual cylinder length=0.3192604814356006 radius=0.4691899845299726
- added link 13, mass 0.15762616033790156; collision cylinder length=0.3192604814356006 radius=0.4691899845299726; visual cylinder length=0.3192604814356006 radius=0.4691899845299726
- added link 14, mass 0.15762616033790156; collision cylinder length=0.3192604814356006 radius=0.4691899845299726; visual cylinder length=0.3192604814356006 radius=0.4691899845299726
- link 0: mass 0.23407871841241357 -> -0.041928476734819975; geometry collision cylinder length=0.21275301331532537 radius=0.6738214328149634; visual cylinder length=0.21275301331532537 radius=0.6738214328149634
- link 11: mass 0.4083755482210827 -> 0.15762616033790156; geometry collision cylinder length=0.3192604814356006 radius=0.4691899845299726; visual cylinder length=0.3192604814356006 radius=0.4691899845299726
Joints:
- removed joint 0_to_22
- removed joint 0_to_23
- removed joint 0_to_24
- added joint 0_to_12: type revolute, parent 0, child 12, origin xyz=0.9131297020884191 0.7471783354347086 0.5441474394424531 rpy=15.357798269208457 2.851366780098196 1.0995151100160443, axis 1 0 0, limit effort=1 velocity=1
- added joint 0_to_13: type revolute, parent 0, child 13, origin xyz=0.9131297020884191 0.7471783354347086 0.5441474394424531 rpy=20.47706435894461 2.851366780098196 1.0995151100160443, axis 1 0 0, limit effort=1 velocity=1
- added joint 0_to_14: type revolute, parent 0, child 14, origin xyz=0.9131297020884191 0.7471783354347086 0.5441474394424531 rpy=25.59633044868076 2.851366780098196 1.0995151100160443, axis 1 0 0, limit effort=1 velocity=1
- joint 0_to_11: origin xyz=0.5711361873981222 0.06355420971682557 0.8084972414942933 rpy=5.957113464629277 1.1621065363046357 5.3823881901385535 -> xyz=0.9131297020884191 0.7471783354347086 0.5441474394424531 rpy=10.238532179472305 2.851366780098196 1.0995151100160443; type fixed -> revolute

File: URDF/10.urdf (robot description, URDF)
Before this commit: robot ted, 7 links, 6 joints
Links:
- removed link 13
- removed link 15
- removed link 24
- removed link 26
- added link 23, mass 0.674776319926726; collision cylinder length=0.43050715634404757 radius=0.9222927091926632; visual cylinder length=0.43050715634404757 radius=0.9222927091926632
- link 0: mass 0.15993937193236452 -> 0.9576674501473837; geometry collision cylinder length=0.6796474057055067 radius=0.06025397025807688; visual cylinder length=0.6796474057055067 radius=0.06025397025807688
- link 11: mass 0.6747531513622993 -> 0.19260508477109606; geometry collision cylinder length=0.5104161326526147 radius=0.36796013857319376; visual cylinder length=0.5104161326526147 radius=0.36796013857319376
- link 22: mass 0.9561266460267444 -> 0.674776319926726; geometry collision cylinder length=0.43050715634404757 radius=0.9222927091926632; visual cylinder length=0.43050715634404757 radius=0.9222927091926632
Joints:
- removed joint 0_to_13
- removed joint 0_to_15
- removed joint 11_to_22
- removed joint 13_to_24
- removed joint 15_to_26
- added joint 0_to_22: type revolute, parent 0, child 22, origin xyz=0.704286072567229 0.8285736280829977 0.45542272978667697 rpy=0.599829968856161 5.251168708810052 4.146831047012167, axis 1 0 0, limit effort=1 velocity=1
- added joint 0_to_23: type revolute, parent 0, child 23, origin xyz=0.704286072567229 0.8285736280829977 0.45542272978667697 rpy=0.7997732918082147 5.251168708810052 4.146831047012167, axis 1 0 0, limit effort=1 velocity=1
- joint 0_to_11: origin xyz=0.4101654414716812 0.5253715872288691 0.7782144858966138 rpy=8.178250881378734 5.490855656101748 0.4532833983370268 -> xyz=0.0647123763930777 0.7159752044118834 0.7679146475609268 rpy=6.045929688295032 5.215080526362034 5.332975148900843

File: URDF/11.urdf (robot description, URDF)
Before this commit: robot ted, 4 links, 3 joints
Links:
- removed link 22
- added link 12, mass 0.9059602521731824; collision cylinder length=0.9549618377048786 radius=0.6301403256943768; visual cylinder length=0.9549618377048786 radius=0.6301403256943768
- added link 24, mass 0.44736366272009565; collision cylinder length=0.8894506098643382 radius=0.7559789026076871; visual cylinder length=0.8894506098643382 radius=0.7559789026076871
- added link 25, mass 0.44736366272009565; collision cylinder length=0.8894506098643382 radius=0.7559789026076871; visual cylinder length=0.8894506098643382 radius=0.7559789026076871
- link 0: mass 0.7706508026362331 -> 0.7457402298794583; geometry collision cylinder length=0.6837529258832584 radius=0.9458604627998224; visual cylinder length=0.6837529258832584 radius=0.9458604627998224
- link 11: mass 0.8568659610022978 -> 0.9059602521731824; geometry collision cylinder length=0.9549618377048786 radius=0.6301403256943768; visual cylinder length=0.9549618377048786 radius=0.6301403256943768
- link 23: mass 0.6075719086087558 -> 0.44736366272009565; geometry collision cylinder length=0.8894506098643382 radius=0.7559789026076871; visual cylinder length=0.8894506098643382 radius=0.7559789026076871
Joints:
- removed joint 0_to_22
- added joint 0_to_12: type revolute, parent 0, child 12, origin xyz=0.3932748374880398 0.616263810309897 0.15444660257576093 rpy=14.446948521983954 0.5170502488772097 3.5920418865609864, axis 1 0 0, limit effort=1 velocity=1
- added joint 0_to_24: type fixed, parent 0, child 24, origin xyz=0.723265815982453 0.879537257236429 0.7359739094194797 rpy=28.61679148780375 4.694204409711059 0.8944217081213673, axis 1 0 0, limit effort=1 velocity=1
- added joint 0_to_25: type fixed, parent 0, child 25, origin xyz=0.723265815982453 0.879537257236429 0.7359739094194797 rpy=34.340149785364495 4.694204409711059 0.8944217081213673, axis 1 0 0, limit effort=1 velocity=1
- joint 0_to_11: origin xyz=0.7741562164640292 0.48507474038404597 0.577923795406728 rpy=4.586103516151838 4.549414251395375 0.5346246509624677 -> xyz=0.3932748374880398 0.616263810309897 0.15444660257576093 rpy=9.63129901465597 0.5170502488772097 3.5920418865609864
- joint 0_to_23: origin xyz=0.4769501562542764 0.707279532225607 0.20012083186896712 rpy=4.675545561369923 0.6988158302917657 3.0689953436694184 -> xyz=0.723265815982453 0.879537257236429 0.7359739094194797 rpy=22.893433190242998 4.694204409711059 0.8944217081213673; type revolute -> fixed

File: URDF/2.urdf (robot description, URDF)
Before this commit: robot ted, 9 links, 8 joints
Links:
- removed link 14
- removed link 25
- removed link 26
- removed link 27
- removed link 28
- link 0: mass 0.46066775353622313 -> -0.041928476734819975; geometry collision cylinder length=0.21275301331532537 radius=0.6738214328149634; visual cylinder length=0.21275301331532537 radius=0.6738214328149634
- link 11: mass 0.02649475875294538 -> 0.11888556824783847; geometry collision cylinder length=0.20148864524368926 radius=0.39336189641222474; visual cylinder length=0.20148864524368926 radius=0.39336189641222474
- link 12: mass 0.02649475875294538 -> 0.11888556824783847; geometry collision cylinder length=0.20148864524368926 radius=0.39336189641222474; visual cylinder length=0.20148864524368926 radius=0.39336189641222474
- link 13: mass 0.02649475875294538 -> 0.11888556824783847; geometry collision cylinder length=0.20148864524368926 radius=0.39336189641222474; visual cylinder length=0.20148864524368926 radius=0.39336189641222474
Joints:
- removed joint 0_to_14
- removed joint 0_to_25
- removed joint 0_to_26
- removed joint 0_to_27
- removed joint 0_to_28
- joint 0_to_11: origin xyz=0.07032620838734782 0.7247642311892147 0.3969425369952374 rpy=3.4866270233156262 3.1845115729762425 1.870276071862189 -> xyz=0.8406967620585992 0.17178042112934833 0.5677756171937046 rpy=1.0264651742255158 2.8809326456153213 2.0432824326917585
- joint 0_to_12: origin xyz=0.07032620838734782 0.7247642311892147 0.3969425369952374 rpy=5.229940534973439 3.1845115729762425 1.870276071862189 -> xyz=0.8406967620585992 0.17178042112934833 0.5677756171937046 rpy=1.5396977613382736 2.8809326456153213 2.0432824326917585
- joint 0_to_13: origin xyz=0.07032620838734782 0.7247642311892147 0.3969425369952374 rpy=6.9732540466312525 3.1845115729762425 1.870276071862189 -> xyz=0.8406967620585992 0.17178042112934833 0.5677756171937046 rpy=2.0529303484510315 2.8809326456153213 2.0432824326917585

File: URDF/3.urdf (robot description, URDF)
Before this commit: robot ted, 16 links, 15 joints
Links:
- removed link 111
- removed link 16
- removed link 210
- removed link 212
- removed link 213
- removed link 214
- removed link 215
- removed link 22
- removed link 23
- removed link 24
- removed link 25
- removed link 27
- removed link 28
- removed link 29
- added link 12, mass 0.2981004832122979; collision cylinder length=0.4067374133161399 radius=0.30882784430971055; visual cylinder length=0.4067374133161399 radius=0.30882784430971055
- added link 13, mass 0.2981004832122979; collision cylinder length=0.4067374133161399 radius=0.30882784430971055; visual cylinder length=0.4067374133161399 radius=0.30882784430971055
- link 0: mass 0.3504002401598274 -> 0.11888556824783847; geometry collision cylinder length=0.20148864524368926 radius=0.39336189641222474; visual cylinder length=0.20148864524368926 radius=0.39336189641222474
- link 11: mass 0.42143478416734315 -> 0.2981004832122979; geometry collision cylinder length=0.4067374133161399 radius=0.30882784430971055; visual cylinder length=0.4067374133161399 radius=0.30882784430971055
Joints:
- removed joint 0_to_111
- removed joint 0_to_16
- removed joint 111_to_212
- removed joint 111_to_213
- removed joint 111_to_214
- removed joint 111_to_215
- removed joint 11_to_22
- removed joint 11_to_23
- removed joint 11_to_24
- removed joint 11_to_25
- removed joint 16_to_210
- removed joint 16_to_27
- removed joint 16_to_28
- removed joint 16_to_29
- added joint 0_to_12: type fixed, parent 0, child 12, origin xyz=0.1813997673060237 0.8592562662678792 0.09256419631250323 rpy=15.220780193260468 1.9793424562395197 0.2541950329481512, axis 1 0 0, limit effort=1 velocity=1
- added joint 0_to_13: type fixed, parent 0, child 13, origin xyz=0.1813997673060237 0.8592562662678792 0.09256419631250323 rpy=20.294373591013958 1.9793424562395197 0.2541950329481512, axis 1 0 0, limit effort=1 velocity=1
- joint 0_to_11: origin xyz=0.22053987618566806 0.11791418867024372 0.23443846621962516 rpy=8.902146545721475 1.9277776971095466 5.8172402069666 -> xyz=0.1813997673060237 0.8592562662678792 0.09256419631250323 rpy=10.147186795506979 1.9793424562395197 0.2541950329481512; type revolute -> fixed

File: URDF/4.urdf (robot description, URDF)
Before this commit: robot ted, 6 links, 5 joints
Links:
- removed link 11
- removed link 22
- removed link 23
- removed link 24
- removed link 25
- link 0: mass 0.14180934674196166 -> -0.041928476734819975; geometry collision cylinder length=0.21275301331532537 radius=0.6738214328149634; visual cylinder length=0.21275301331532537 radius=0.6738214328149634
Joints:
- removed joint 0_to_11
- removed joint 0_to_22
- removed joint 0_to_23
- removed joint 0_to_24
- removed joint 0_to_25

File: URDF/5.urdf (robot description, URDF)
Before this commit: robot ted, 5 links, 4 joints
Links:
- removed link 22
- removed link 23
- added link 12, mass 0.11888556824783847; collision cylinder length=0.20148864524368926 radius=0.39336189641222474; visual cylinder length=0.20148864524368926 radius=0.39336189641222474
- added link 13, mass 0.11888556824783847; collision cylinder length=0.20148864524368926 radius=0.39336189641222474; visual cylinder length=0.20148864524368926 radius=0.39336189641222474
- added link 25, mass 0.21899950248364408; collision cylinder length=0.6914661831663674 radius=0.8007755610867969; visual cylinder length=0.6914661831663674 radius=0.8007755610867969
- link 0: mass 0.5915219888699443 -> -0.041928476734819975; geometry collision cylinder length=0.30804062851760383 radius=0.6738214328149634; visual cylinder length=0.30804062851760383 radius=0.6738214328149634
- link 11: mass 0.5587351277461894 -> 0.11888556824783847; geometry collision cylinder length=0.20148864524368926 radius=0.39336189641222474; visual cylinder length=0.20148864524368926 radius=0.39336189641222474
- link 24: mass 0.5927891381067416 -> 0.21899950248364408; geometry collision cylinder length=0.6914661831663674 radius=0.8007755610867969; visual cylinder length=0.6914661831663674 radius=0.8007755610867969
Joints:
- removed joint 11_to_22
- removed joint 11_to_23
- removed joint 11_to_24
- added joint 0_to_12: type revolute, parent 0, child 12, origin xyz=0.8406967620585992 0.17178042112934833 0.5677756171937046 rpy=1.5396977613382736 2.8809326456153213 2.0432824326917585, axis 1 0 0, limit effort=1 velocity=1
- added joint 0_to_13: type revolute, parent 0, child 13, origin xyz=0.8406967620585992 0.17178042112934833 0.5677756171937046 rpy=2.0529303484510315 2.8809326456153213 2.0432824326917585, axis 1 0 0, limit effort=1 velocity=1
- added joint 0_to_24: type revolute, parent 0, child 24, origin xyz=0.6393194556138254 0.591008357849777 0.6075456806105207 rpy=8.195870269966074 0.5896338279879213 6.0474511397840685, axis 1 0 0, limit effort=1 velocity=1
- added joint 0_to_25: type revolute, parent 0, child 25, origin xyz=0.6393194556138254 0.591008357849777 0.6075456806105207 rpy=9.835044323959288 0.5896338279879213 6.0474511397840685, axis 1 0 0, limit effort=1 velocity=1
- joint 0_to_11: origin xyz=0.9523668133272517 0.44254823454720327 0.25603083030857443 rpy=12.5325441779656 4.158678781984297 2.503122342430801 -> xyz=0.8406967620585992 0.17178042112934833 0.5677756171937046 rpy=1.0264651742255158 2.8809326456153213 2.0432824326917585; type fixed -> revolute

File: URDF/6.urdf (robot description, URDF)
Before this commit: robot ted, 10 links, 9 joints
Links:
- removed link 11
- removed link 14
- removed link 17
- removed link 22
- removed link 23
- removed link 25
- removed link 26
- removed link 28
- removed link 29
- link 0: mass 0.9416563593579919 -> -0.041928476734819975; geometry collision cylinder length=0.21275301331532537 radius=0.6738214328149634; visual cylinder length=0.21275301331532537 radius=0.6738214328149634
Joints:
- removed joint 0_to_11
- removed joint 0_to_14
- removed joint 0_to_17
- removed joint 11_to_22
- removed joint 11_to_23
- removed joint 14_to_25
- removed joint 14_to_26
- removed joint 17_to_28
- removed joint 17_to_29

File: URDF/7.urdf (robot description, URDF)
Before this commit: robot ted, 7 links, 6 joints
Links:
- removed link 14
- removed link 25
- removed link 26
- added link 24, mass 0.19156958755707632; collision cylinder length=0.13915390401645178 radius=0.0363710677609137; visual cylinder length=0.13915390401645178 radius=0.0363710677609137
- link 0: mass 0.05787979911680308 -> -0.041928476734819975; geometry collision cylinder length=0.21275301331532537 radius=0.6738214328149634; visual cylinder length=0.21275301331532537 radius=0.6738214328149634
- link 11: mass 0.4053506420887715 -> 0.11888556824783847; geometry collision cylinder length=0.20148864524368926 radius=0.39336189641222474; visual cylinder length=0.20148864524368926 radius=0.39336189641222474
- link 12: mass 0.4053506420887715 -> 0.11888556824783847; geometry collision cylinder length=0.20148864524368926 radius=0.39336189641222474; visual cylinder length=0.20148864524368926 radius=0.39336189641222474
- link 13: mass 0.4053506420887715 -> 0.11888556824783847; geometry collision cylinder length=0.20148864524368926 radius=0.39336189641222474; visual cylinder length=0.20148864524368926 radius=0.39336189641222474
Joints:
- removed joint 0_to_14
- removed joint 0_to_25
- removed joint 0_to_26
- added joint 0_to_24: type revolute, parent 0, child 24, origin xyz=0.6737033473129543 0.5669926058583141 0.612682514354474 rpy=9.851719949138007 5.838098258830235 1.4353374141715116, axis 1 0 0, limit effort=1 velocity=1
- joint 0_to_11: origin xyz=0.24242234705389487 0.33828020878731035 0.2959242856990707 rpy=5.377656601893495 4.32067423514443 3.563202333276369 -> xyz=0.8406967620585992 0.17178042112934833 0.5677756171937046 rpy=1.0264651742255158 2.8809326456153213 2.0432824326917585
- joint 0_to_12: origin xyz=0.24242234705389487 0.33828020878731035 0.2959242856990707 rpy=8.066484902840243 4.32067423514443 3.563202333276369 -> xyz=0.8406967620585992 0.17178042112934833 0.5677756171937046 rpy=1.5396977613382736 2.8809326456153213 2.0432824326917585
- joint 0_to_13: origin xyz=0.24242234705389487 0.33828020878731035 0.2959242856990707 rpy=10.75531320378699 4.32067423514443 3.563202333276369 -> xyz=0.8406967620585992 0.17178042112934833 0.5677756171937046 rpy=2.0529303484510315 2.8809326456153213 2.0432824326917585

File: URDF/8.urdf (robot description, URDF)
Before this commit: robot ted, 4 links, 3 joints
Links:
- removed link 22
- removed link 23
- added link 12, mass 0.11888556824783847; collision cylinder length=0.20148864524368926 radius=0.39336189641222474; visual cylinder length=0.20148864524368926 radius=0.39336189641222474
- added link 13, mass 0.11888556824783847; collision cylinder length=0.20148864524368926 radius=0.39336189641222474; visual cylinder length=0.20148864524368926 radius=0.39336189641222474
- link 0: mass 0.918851376352353 -> -0.041928476734819975; geometry collision cylinder length=0.21275301331532537 radius=0.6738214328149634; visual cylinder length=0.21275301331532537 radius=0.6738214328149634
- link 11: mass 0.5869899911583579 -> 0.11888556824783847; geometry collision cylinder length=0.20148864524368926 radius=0.39336189641222474; visual cylinder length=0.20148864524368926 radius=0.39336189641222474
Joints:
- removed joint 11_to_22
- removed joint 11_to_23
- added joint 0_to_12: type revolute, parent 0, child 12, origin xyz=0.8406967620585992 0.17178042112934833 0.5677756171937046 rpy=1.5396977613382736 2.8809326456153213 2.0432824326917585, axis 1 0 0, limit effort=1 velocity=1
- added joint 0_to_13: type revolute, parent 0, child 13, origin xyz=0.8406967620585992 0.17178042112934833 0.5677756171937046 rpy=2.0529303484510315 2.8809326456153213 2.0432824326917585, axis 1 0 0, limit effort=1 velocity=1
- joint 0_to_11: origin xyz=0.31356293640167177 0.7714657555208229 0.746370997194334 rpy=12.367558002888956 0.367235277655106 4.608598057269663 -> xyz=0.8406967620585992 0.17178042112934833 0.5677756171937046 rpy=1.0264651742255158 2.8809326456153213 2.0432824326917585

File: URDF/9.urdf (robot description, URDF)
Before this commit: robot ted, 4 links, 3 joints
Links:
- removed link 11
- removed link 12
- removed link 23
- link 0: mass 0.5727515049594439 -> -0.041928476734819975; geometry collision cylinder length=0.21275301331532537 radius=0.6738214328149634; visual cylinder length=0.21275301331532537 radius=0.6738214328149634
Joints:
- removed joint 0_to_11
- removed joint 0_to_12
- removed joint 0_to_23

File: URDF/test.urdf (robot description, URDF)
Before this commit: robot ted, 9 links, 8 joints
Links:
- removed link 23
- removed link 24
- removed link 35
- removed link 36
- removed link 37
- removed link 38
- removed link 42
- added link 12, mass 0.11888556824783847; collision cylinder length=0.20148864524368926 radius=0.39336189641222474; visual cylinder length=0.20148864524368926 radius=0.39336189641222474
- added link 13, mass 0.11888556824783847; collision cylinder length=0.20148864524368926 radius=0.39336189641222474; visual cylinder length=0.20148864524368926 radius=0.39336189641222474
- link 0: mass 0.11648996513674648 -> -0.041928476734819975; geometry collision cylinder length=0.21275301331532537 radius=0.6738214328149634; visual cylinder length=0.21275301331532537 radius=0.6738214328149634
- link 11: mass 0.3523990213604573 -> 0.11888556824783847; geometry collision cylinder length=0.20148864524368926 radius=0.39336189641222474; visual cylinder length=0.20148864524368926 radius=0.39336189641222474
Joints:
- removed joint 0_to_23
- removed joint 0_to_24
- removed joint 0_to_35
- removed joint 0_to_36
- removed joint 0_to_37
- removed joint 0_to_38
- removed joint 11_to_42
- added joint 0_to_12: type revolute, parent 0, child 12, origin xyz=0.8406967620585992 0.17178042112934833 0.5677756171937046 rpy=1.5396977613382736 2.8809326456153213 2.0432824326917585, axis 1 0 0, limit effort=1 velocity=1
- added joint 0_to_13: type revolute, parent 0, child 13, origin xyz=0.8406967620585992 0.17178042112934833 0.5677756171937046 rpy=2.0529303484510315 2.8809326456153213 2.0432824326917585, axis 1 0 0, limit effort=1 velocity=1
- joint 0_to_11: origin xyz=0.09165277779681158 0.13365902240918626 0.9638148957205093 rpy=5.447595852843178 0.05992295207809395 2.8285596048779307 -> xyz=0.8406967620585992 0.17178042112934833 0.5677756171937046 rpy=1.0264651742255158 2.8809326456153213 2.0432824326917585
