Commit message: starting hyper-parameter testing

File: URDF/0.urdf (robot description, URDF)
Before this commit: robot ted, 4 links, 3 joints
Links:
- removed link 12
- removed link 13
- added link 15, mass 0.21962730422956667; collision cylinder length=0.32768364753998247 radius=0.6765220306374614; visual cylinder length=0.32768364753998247 radius=0.6765220306374614
- added link 22, mass 0.41090573523269014; collision cylinder length=0.5895765108887729 radius=0.607391736853669; visual cylinder length=0.5895765108887729 radius=0.607391736853669
- added link 23, mass 0.41090573523269014; collision cylinder length=0.5895765108887729 radius=0.607391736853669; visual cylinder length=0.5895765108887729 radius=0.607391736853669
- added link 24, mass 0.41090573523269014; collision cylinder length=0.5895765108887729 radius=0.607391736853669; visual cylinder length=0.5895765108887729 radius=0.607391736853669
- added link 26, mass 0.41090573523269014; collision cylinder length=0.5895765108887729 radius=0.607391736853669; visual cylinder length=0.5895765108887729 radius=0.607391736853669
- added link 27, mass 0.41090573523269014; collision cylinder length=0.5895765108887729 radius=0.607391736853669; visual cylinder length=0.5895765108887729 radius=0.607391736853669
- added link 28, mass 0.41090573523269014; collision cylinder length=0.5895765108887729 radius=0.607391736853669; visual cylinder length=0.5895765108887729 radius=0.607391736853669
- link 0: mass -0.041928476734819975 -> 0.6406075354898184; geometry collision cylinder length=0.15113824252047015 radius=0.4296970259490408; visual cylinder length=0.15113824252047015 radius=0.4296970259490408
- link 11: mass 0.11888556824783847 -> 0.21962730422956667; geometry collision cylinder length=0.32768364753998247 radius=0.6765220306374614; visual cylinder length=0.32768364753998247 radius=0.6765220306374614
Joints:
- removed joint 0_to_12
- removed joint 0_to_13
- added joint 0_to_15: type revolute, parent 0, child 15, origin xyz=0.41173728907590745 0.7121282447210531 0.5824931766248451 rpy=14.658880708369878 6.135237077640203 4.673844728901479, axis 1 0 0, limit effort=1 velocity=1
- added joint 11_to_22: type revolute, parent 11, child 22, origin xyz=0.953866148735442 0.6548537646260819 0.11013515940345642 rpy=2.102332137072244 1.5801231317912616 6.119977702978318, axis 1 0 0, limit effort=1 velocity=1
- added joint 11_to_23: type revolute, parent 11, child 23, origin xyz=0.953866148735442 0.6548537646260819 0.11013515940345642 rpy=3.153498205608366 1.5801231317912616 6.119977702978318, axis 1 0 0, limit effort=1 velocity=1
- added joint 11_to_24: type revolute, parent 11, child 24, origin xyz=0.953866148735442 0.6548537646260819 0.11013515940345642 rpy=4.204664274144488 1.5801231317912616 6.119977702978318, axis 1 0 0, limit effort=1 velocity=1
- added joint 15_to_26: type revolute, parent 15, child 26, origin xyz=0.953866148735442 0.6548537646260819 0.11013515940345642 rpy=2.102332137072244 1.5801231317912616 6.119977702978318, axis 1 0 0, limit effort=1 velocity=1
- added joint 15_to_27: type revolute, parent 15, child 27, origin xyz=0.953866148735442 0.6548537646260819 0.11013515940345642 rpy=3.153498205608366 1.5801231317912616 6.119977702978318, axis 1 0 0, limit effort=1 velocity=1
- added joint 15_to_28: type revolute, parent 15, child 28, origin xyz=0.953866148735442 0.6548537646260819 0.11013515940345642 rpy=4.204664274144488 1.5801231317912616 6.119977702978318, axis 1 0 0, limit effort=1 velocity=1
- joint 0_to_11: origin xyz=0.8406967620585992 0.17178042112934833 0.5677756171937046 rpy=1.0264651742255158 2.8809326456153213 2.0432824326917585 -> xyz=0.41173728907590745 0.7121282447210531 0.5824931766248451 rpy=9.772587138913252 6.135237077640203 4.673844728901479

File: URDF/1.urdf (robot description, URDF)
Before this commit: robot ted, 5 links, 4 joints
Links:
- removed link 12
- removed link 13
- removed link 14
- added link 15, mass 0.21962730422956667; collision cylinder length=0.32768364753998247 radius=0.6765220306374614; visual cylinder length=0.32768364753998247 radius=0.6765220306374614
- added link 22, mass 0.41090573523269014; collision cylinder length=0.5895765108887729 radius=0.607391736853669; visual cylinder length=0.5895765108887729 radius=0.607391736853669
- added link 23, mass 0.41090573523269014; collision cylinder length=0.5895765108887729 radius=0.607391736853669; visual cylinder length=0.5895765108887729 radius=0.607391736853669
- added link 24, mass 0.41090573523269014; collision cylinder length=0.5895765108887729 radius=0.607391736853669; visual cylinder length=0.5895765108887729 radius=0.607391736853669
- added link 26, mass 0.41090573523269014; collision cylinder length=0.5895765108887729 radius=0.607391736853669; visual cylinder length=0.5895765108887729 radius=0.607391736853669
- added link 27, mass 0.41090573523269014; collision cylinder length=0.5895765108887729 radius=0.607391736853669; visual cylinder length=0.5895765108887729 radius=0.607391736853669
- added link 28, mass 0.41090573523269014; collision cylinder length=0.5895765108887729 radius=0.607391736853669; visual cylinder length=0.5895765108887729 radius=0.607391736853669
- link 0: mass -0.041928476734819975 -> 0.6406075354898184; geometry collision cylinder length=0.15113824252047015 radius=0.4296970259490408; visual cylinder length=0.15113824252047015 radius=0.4296970259490408
- link 11: mass 0.15762616033790156 -> 0.21962730422956667; geometry collision cylinder length=0.32768364753998247 radius=0.6765220306374614; visual cylinder length=0.32768364753998247 radius=0.6765220306374614
Joints:
- removed joint 0_to_12
- removed joint 0_to_13
- removed joint 0_to_14
- added joint 0_to_15: type revolute, parent 0, child 15, origin xyz=0.41173728907590745 0.7121282447210531 0.5824931766248451 rpy=14.658880708369878 6.135237077640203 4.673844728901479, axis 1 0 0, limit effort=1 velocity=1
- added joint 11_to_22: type revolute, parent 11, child 22, origin xyz=0.953866148735442 0.6548537646260819 0.11013515940345642 rpy=2.102332137072244 1.5801231317912616 6.119977702978318, axis 1 0 0, limit effort=1 velocity=1
- added joint 11_to_23: type revolute, parent 11, child 23, origin xyz=0.953866148735442 0.6548537646260819 0.11013515940345642 rpy=3.153498205608366 1.5801231317912616 6.119977702978318, axis 1 0 0, limit effort=1 velocity=1
- added joint 11_to_24: type revolute, parent 11, child 24, origin xyz=0.953866148735442 0.6548537646260819 0.11013515940345642 rpy=4.204664274144488 1.5801231317912616 6.119977702978318, axis 1 0 0, limit effort=1 velocity=1
- added joint 15_to_26: type revolute, parent 15, child 26, origin xyz=0.953866148735442 0.6548537646260819 0.11013515940345642 rpy=2.102332137072244 1.5801231317912616 6.119977702978318, axis 1 0 0, limit effort=1 velocity=1
- added joint 15_to_27: type revolute, parent 15, child 27, origin xyz=0.953866148735442 0.6548537646260819 0.11013515940345642 rpy=3.153498205608366 1.5801231317912616 6.119977702978318, axis 1 0 0, limit effort=1 velocity=1
- added joint 15_to_28: type revolute, parent 15, child 28, origin xyz=0.953866148735442 0.6548537646260819 0.11013515940345642 rpy=4.204664274144488 1.5801231317912616 6.119977702978318, axis 1 0 0, limit effort=1 velocity=1
- joint 0_to_11: origin xyz=0.9131297020884191 0.7471783354347086 0.5441474394424531 rpy=10.238532179472305 2.851366780098196 1.0995151100160443 -> xyz=0.41173728907590745 0.7121282447210531 0.5824931766248451 rpy=9.772587138913252 6.135237077640203 4.673844728901479

File: URDF/3.urdf (robot description, URDF)
Before this commit: robot ted, 4 links, 3 joints
Links:
- removed link 12
- removed link 13
- added link 15, mass 0.21962730422956667; collision cylinder length=0.32768364753998247 radius=0.6765220306374614; visual cylinder length=0.32768364753998247 radius=0.6765220306374614
- added link 22, mass 0.41090573523269014; collision cylinder length=0.5895765108887729 radius=0.607391736853669; visual cylinder length=0.5895765108887729 radius=0.607391736853669
- added link 23, mass 0.41090573523269014; collision cylinder length=0.5895765108887729 radius=0.607391736853669; visual cylinder length=0.5895765108887729 radius=0.607391736853669
- added link 24, mass 0.41090573523269014; collision cylinder length=0.5895765108887729 radius=0.607391736853669; visual cylinder length=0.5895765108887729 radius=0.607391736853669
- added link 26, mass 0.41090573523269014; collision cylinder length=0.5895765108887729 radius=0.607391736853669; visual cylinder length=0.5895765108887729 radius=0.607391736853669
- added link 27, mass 0.41090573523269014; collision cylinder length=0.5895765108887729 radius=0.607391736853669; visual cylinder length=0.5895765108887729 radius=0.607391736853669
- added link 28, mass 0.41090573523269014; collision cylinder length=0.5895765108887729 radius=0.607391736853669; visual cylinder length=0.5895765108887729 radius=0.607391736853669
- link 0: mass 0.11888556824783847 -> 0.6406075354898184; geometry collision cylinder length=0.15113824252047015 radius=0.4296970259490408; visual cylinder length=0.15113824252047015 radius=0.4296970259490408
- link 11: mass 0.2981004832122979 -> 0.21962730422956667; geometry collision cylinder length=0.32768364753998247 radius=0.6765220306374614; visual cylinder length=0.32768364753998247 radius=0.6765220306374614
Joints:
- removed joint 0_to_12
- removed joint 0_to_13
- added joint 0_to_15: type revolute, parent 0, child 15, origin xyz=0.41173728907590745 0.7121282447210531 0.5824931766248451 rpy=14.658880708369878 6.135237077640203 4.673844728901479, axis 1 0 0, limit effort=1 velocity=1
- added joint 11_to_22: type revolute, parent 11, child 22, origin xyz=0.953866148735442 0.6548537646260819 0.11013515940345642 rpy=2.102332137072244 1.5801231317912616 6.119977702978318, axis 1 0 0, limit effort=1 velocity=1
- added joint 11_to_23: type revolute, parent 11, child 23, origin xyz=0.953866148735442 0.6548537646260819 0.11013515940345642 rpy=3.153498205608366 1.5801231317912616 6.119977702978318, axis 1 0 0, limit effort=1 velocity=1
- added joint 11_to_24: type revolute, parent 11, child 24, origin xyz=0.953866148735442 0.6548537646260819 0.11013515940345642 rpy=4.204664274144488 1.5801231317912616 6.119977702978318, axis 1 0 0, limit effort=1 velocity=1
- added joint 15_to_26: type revolute, parent 15, child 26, origin xyz=0.953866148735442 0.6548537646260819 0.11013515940345642 rpy=2.102332137072244 1.5801231317912616 6.119977702978318, axis 1 0 0, limit effort=1 velocity=1
- added joint 15_to_27: type revolute, parent 15, child 27, origin xyz=0.953866148735442 0.6548537646260819 0.11013515940345642 rpy=3.153498205608366 1.5801231317912616 6.119977702978318, axis 1 0 0, limit effort=1 velocity=1
- added joint 15_to_28: type revolute, parent 15, child 28, origin xyz=0.953866148735442 0.6548537646260819 0.11013515940345642 rpy=4.204664274144488 1.5801231317912616 6.119977702978318, axis 1 0 0, limit effort=1 velocity=1
- joint 0_to_11: origin xyz=0.1813997673060237 0.8592562662678792 0.09256419631250323 rpy=10.147186795506979 1.9793424562395197 0.2541950329481512 -> xyz=0.41173728907590745 0.7121282447210531 0.5824931766248451 rpy=9.772587138913252 6.135237077640203 4.673844728901479; type fixed -> revolute

File: URDF/4.urdf (robot description, URDF)
Before this commit: robot ted, 1 links, 0 joints
Links:
- added link 11, mass 0.21962730422956667; collision cylinder length=0.32768364753998247 radius=0.6765220306374614; visual cylinder length=0.32768364753998247 radius=0.6765220306374614
- added link 15, mass 0.21962730422956667; collision cylinder length=0.32768364753998247 radius=0.6765220306374614; visual cylinder length=0.32768364753998247 radius=0.6765220306374614
- added link 22, mass 0.41090573523269014; collision cylinder length=0.5895765108887729 radius=0.607391736853669; visual cylinder length=0.5895765108887729 radius=0.607391736853669
- added link 23, mass 0.41090573523269014; collision cylinder length=0.5895765108887729 radius=0.607391736853669; visual cylinder length=0.5895765108887729 radius=0.607391736853669
- added link 24, mass 0.41090573523269014; collision cylinder length=0.5895765108887729 radius=0.607391736853669; visual cylinder length=0.5895765108887729 radius=0.607391736853669
- added link 26, mass 0.41090573523269014; collision cylinder length=0.5895765108887729 radius=0.607391736853669; visual cylinder length=0.5895765108887729 radius=0.607391736853669
- added link 27, mass 0.41090573523269014; collision cylinder length=0.5895765108887729 radius=0.607391736853669; visual cylinder length=0.5895765108887729 radius=0.607391736853669
- added link 28, mass 0.41090573523269014; collision cylinder length=0.5895765108887729 radius=0.607391736853669; visual cylinder length=0.5895765108887729 radius=0.607391736853669
- link 0: mass -0.041928476734819975 -> 0.6406075354898184; geometry collision cylinder length=0.15113824252047015 radius=0.4296970259490408; visual cylinder length=0.15113824252047015 radius=0.4296970259490408
Joints:
- added joint 0_to_11: type revolute, parent 0, child 11, origin xyz=0.41173728907590745 0.7121282447210531 0.5824931766248451 rpy=9.772587138913252 6.135237077640203 4.455457061760032, axis 1 0 0, limit effort=1 velocity=1
- added joint 0_to_15: type revolute, parent 0, child 15, origin xyz=0.41173728907590745 0.7121282447210531 0.5824931766248451 rpy=14.658880708369878 6.135237077640203 4.455457061760032, axis 1 0 0, limit effort=1 velocity=1
- added joint 11_to_22: type revolute, parent 11, child 22, origin xyz=0.953866148735442 0.6548537646260819 0.11013515940345642 rpy=2.102332137072244 1.5801231317912616 6.119977702978318, axis 1 0 0, limit effort=1 velocity=1
- added joint 11_to_23: type revolute, parent 11, child 23, origin xyz=0.953866148735442 0.6548537646260819 0.11013515940345642 rpy=3.153498205608366 1.5801231317912616 6.119977702978318, axis 1 0 0, limit effort=1 velocity=1
- added joint 11_to_24: type revolute, parent 11, child 24, origin xyz=0.953866148735442 0.6548537646260819 0.11013515940345642 rpy=4.204664274144488 1.5801231317912616 6.119977702978318, axis 1 0 0, limit effort=1 velocity=1
- added joint 15_to_26: type revolute, parent 15, child 26, origin xyz=0.953866148735442 0.6548537646260819 0.11013515940345642 rpy=2.102332137072244 1.5801231317912616 6.119977702978318, axis 1 0 0, limit effort=1 velocity=1
- added joint 15_to_27: type revolute, parent 15, child 27, origin xyz=0.953866148735442 0.6548537646260819 0.11013515940345642 rpy=3.153498205608366 1.5801231317912616 6.119977702978318, axis 1 0 0, limit effort=1 velocity=1
- added joint 15_to_28: type revolute, parent 15, child 28, origin xyz=0.953866148735442 0.6548537646260819 0.11013515940345642 rpy=4.204664274144488 1.5801231317912616 6.119977702978318, axis 1 0 0, limit effort=1 velocity=1

File: URDF/5.urdf (robot description, URDF)
Before this commit: robot ted, 6 links, 5 joints
Links:
- removed link 12
- removed link 13
- removed link 25
- added link 15, mass 0.21962730422956667; collision cylinder length=0.32768364753998247 radius=0.6765220306374614; visual cylinder length=0.32768364753998247 radius=0.6765220306374614
- added link 22, mass 0.41090573523269014; collision cylinder length=0.5895765108887729 radius=0.607391736853669; visual cylinder length=0.5895765108887729 radius=0.607391736853669
- added link 23, mass 0.41090573523269014; collision cylinder length=0.5895765108887729 radius=0.607391736853669; visual cylinder length=0.5895765108887729 radius=0.607391736853669
- added link 26, mass 0.41090573523269014; collision cylinder length=0.5895765108887729 radius=0.607391736853669; visual cylinder length=0.5895765108887729 radius=0.607391736853669
- added link 27, mass 0.41090573523269014; collision cylinder length=0.5895765108887729 radius=0.607391736853669; visual cylinder length=0.5895765108887729 radius=0.607391736853669
- added link 28, mass 0.41090573523269014; collision cylinder length=0.5895765108887729 radius=0.607391736853669; visual cylinder length=0.5895765108887729 radius=0.607391736853669
- link 0: mass -0.041928476734819975 -> 0.6406075354898184; geometry collision cylinder length=0.15113824252047015 radius=0.4296970259490408; visual cylinder length=0.15113824252047015 radius=0.4296970259490408
- link 11: mass 0.11888556824783847 -> 0.21962730422956667; geometry collision cylinder length=0.32768364753998247 radius=0.6765220306374614; visual cylinder length=0.32768364753998247 radius=0.6765220306374614
- link 24: mass 0.21899950248364408 -> 0.41090573523269014; geometry collision cylinder length=0.5895765108887729 radius=0.607391736853669; visual cylinder length=0.5895765108887729 radius=0.607391736853669
Joints:
- removed joint 0_to_12
- removed joint 0_to_13
- removed joint 0_to_24
- removed joint 0_to_25
- added joint 0_to_15: type revolute, parent 0, child 15, origin xyz=0.41173728907590745 0.7121282447210531 0.5824931766248451 rpy=14.658880708369878 6.135237077640203 4.673844728901479, axis 1 0 0, limit effort=1 velocity=1
- added joint 11_to_22: type revolute, parent 11, child 22, origin xyz=0.953866148735442 0.6548537646260819 0.11013515940345642 rpy=2.102332137072244 1.5801231317912616 6.119977702978318, axis 1 0 0, limit effort=1 velocity=1
- added joint 11_to_23: type revolute, parent 11, child 23, origin xyz=0.953866148735442 0.6548537646260819 0.11013515940345642 rpy=3.153498205608366 1.5801231317912616 6.119977702978318, axis 1 0 0, limit effort=1 velocity=1
- added joint 11_to_24: type revolute, parent 11, child 24, origin xyz=0.953866148735442 0.6548537646260819 0.11013515940345642 rpy=4.204664274144488 1.5801231317912616 6.119977702978318, axis 1 0 0, limit effort=1 velocity=1
- added joint 15_to_26: type revolute, parent 15, child 26, origin xyz=0.953866148735442 0.6548537646260819 0.11013515940345642 rpy=2.102332137072244 1.5801231317912616 6.119977702978318, axis 1 0 0, limit effort=1 velocity=1
- added joint 15_to_27: type revolute, parent 15, child 27, origin xyz=0.953866148735442 0.6548537646260819 0.11013515940345642 rpy=3.153498205608366 1.5801231317912616 6.119977702978318, axis 1 0 0, limit effort=1 velocity=1
- added joint 15_to_28: type revolute, parent 15, child 28, origin xyz=0.953866148735442 0.6548537646260819 0.11013515940345642 rpy=4.204664274144488 1.5801231317912616 6.119977702978318, axis 1 0 0, limit effort=1 velocity=1
- joint 0_to_11: origin xyz=0.8406967620585992 0.17178042112934833 0.5677756171937046 rpy=1.0264651742255158 2.8809326456153213 2.0432824326917585 -> xyz=0.41173728907590745 0.7121282447210531 0.5824931766248451 rpy=9.772587138913252 6.135237077640203 4.673844728901479

File: URDF/6.urdf (robot description, URDF)
Before this commit: robot ted, 1 links, 0 joints
Links:
- added link 11, mass 0.41090573523269014; collision cylinder length=0.5895765108887729 radius=0.607391736853669; visual cylinder length=0.5895765108887729 radius=0.607391736853669
- added link 12, mass 0.41090573523269014; collision cylinder length=0.5895765108887729 radius=0.607391736853669; visual cylinder length=0.5895765108887729 radius=0.607391736853669
- added link 13, mass 0.41090573523269014; collision cylinder length=0.5895765108887729 radius=0.607391736853669; visual cylinder length=0.5895765108887729 radius=0.607391736853669
- link 0: mass -0.041928476734819975 -> 0.6406075354898184; geometry collision cylinder length=0.15113824252047015 radius=0.4296970259490408; visual cylinder length=0.15113824252047015 radius=0.4296970259490408
Joints:
- added joint 0_to_11: type revolute, parent 0, child 11, origin xyz=0.953866148735442 0.6548537646260819 0.11013515940345642 rpy=2.102332137072244 1.5801231317912616 6.119977702978318, axis 1 0 0, limit effort=1 velocity=1
- added joint 0_to_12: type revolute, parent 0, child 12, origin xyz=0.953866148735442 0.6548537646260819 0.11013515940345642 rpy=3.153498205608366 1.5801231317912616 6.119977702978318, axis 1 0 0, limit effort=1 velocity=1
- added joint 0_to_13: type revolute, parent 0, child 13, origin xyz=0.953866148735442 0.6548537646260819 0.11013515940345642 rpy=4.204664274144488 1.5801231317912616 6.119977702978318, axis 1 0 0, limit effort=1 velocity=1

File: URDF/7.urdf (robot description, URDF)
Before this commit: robot ted, 5 links, 4 joints
Links:
- removed link 24
- link 0: mass -0.041928476734819975 -> 0.21962730422956667; geometry collision cylinder length=0.32768364753998247 radius=0.6765220306374614; visual cylinder length=0.32768364753998247 radius=0.6765220306374614
- link 11: mass 0.11888556824783847 -> 0.41090573523269014; geometry collision cylinder length=0.5895765108887729 radius=0.607391736853669; visual cylinder length=0.5895765108887729 radius=0.607391736853669
- link 12: mass 0.11888556824783847 -> 0.41090573523269014; geometry collision cylinder length=0.5895765108887729 radius=0.607391736853669; visual cylinder length=0.5895765108887729 radius=0.607391736853669
- link 13: mass 0.11888556824783847 -> 0.41090573523269014; geometry collision cylinder length=0.5895765108887729 radius=0.607391736853669; visual cylinder length=0.5895765108887729 radius=0.607391736853669
Joints:
- removed joint 0_to_24
- joint 0_to_11: origin xyz=0.8406967620585992 0.17178042112934833 0.5677756171937046 rpy=1.0264651742255158 2.8809326456153213 2.0432824326917585 -> xyz=0.953866148735442 0.6548537646260819 0.11013515940345642 rpy=2.102332137072244 1.5801231317912616 6.119977702978318
- joint 0_to_12: origin xyz=0.8406967620585992 0.17178042112934833 0.5677756171937046 rpy=1.5396977613382736 2.8809326456153213 2.0432824326917585 -> xyz=0.953866148735442 0.6548537646260819 0.11013515940345642 rpy=3.153498205608366 1.5801231317912616 6.119977702978318
- joint 0_to_13: origin xyz=0.8406967620585992 0.17178042112934833 0.5677756171937046 rpy=2.0529303484510315 2.8809326456153213 2.0432824326917585 -> xyz=0.953866148735442 0.6548537646260819 0.11013515940345642 rpy=4.204664274144488 1.5801231317912616 6.119977702978318
