Commit message: starting hyper-parameter testing

File: URDF/9.urdf (robot description, URDF)
Before this commit: robot ted, 1 links, 0 joints
Links:
- added link 11, mass 0.21962730422956667; collision cylinder length=0.32768364753998247 radius=0.6765220306374614; visual cylinder length=0.32768364753998247 radius=0.6765220306374614
- added link 12, mass 0.21962730422956667; collision cylinder length=0.32768364753998247 radius=0.6765220306374614; visual cylinder length=0.32768364753998247 radius=0.6765220306374614
- added link 23, mass 0.949285747241063; collision cylinder length=0.04094705211965233 radius=0.9732910157379706; visual cylinder length=0.04094705211965233 radius=0.9732910157379706
- added link 24, mass 0.949285747241063; collision cylinder length=0.04094705211965233 radius=0.9732910157379706; visual cylinder length=0.04094705211965233 radius=0.9732910157379706
- added link 25, mass 0.949285747241063; collision cylinder length=0.04094705211965233 radius=0.9732910157379706; visual cylinder length=0.04094705211965233 radius=0.9732910157379706
- added link 26, mass 0.949285747241063; collision cylinder length=0.04094705211965233 radius=0.9732910157379706; visual cylinder length=0.04094705211965233 radius=0.9732910157379706
- link 0: mass -0.041928476734819975 -> 0.6406075354898184; geometry collision cylinder length=0.15113824252047015 radius=0.4296970259490408; visual cylinder length=0.15113824252047015 radius=0.4296970259490408
Joints:
- added joint 0_to_11: type revolute, parent 0, child 11, origin xyz=0.41173728907590745 0.7121282447210531 0.5824931766248451 rpy=9.772587138913252 6.135237077640203 4.673844728901479, axis 1 0 0, limit effort=1 velocity=1
- added joint 0_to_12: type revolute, parent 0, child 12, origin xyz=0.41173728907590745 0.7121282447210531 0.5824931766248451 rpy=14.658880708369878 6.135237077640203 4.673844728901479, axis 1 0 0, limit effort=1 velocity=1
- added joint 0_to_23: type revolute, parent 0, child 23, origin xyz=0.09765164843013574 0.20035762048898975 0.11690241594468376 rpy=0.06512036214053042 3.320549569090366 4.698188204105016, axis 1 0 0, limit effort=1 velocity=1
- added joint 0_to_24: type revolute, parent 0, child 24, origin xyz=0.09765164843013574 0.20035762048898975 0.11690241594468376 rpy=0.08140045267566302 3.320549569090366 4.698188204105016, axis 1 0 0, limit effort=1 velocity=1
- added joint 0_to_25: type revolute, parent 0, child 25, origin xyz=0.09765164843013574 0.20035762048898975 0.11690241594468376 rpy=0.09768054321079564 3.320549569090366 4.698188204105016, axis 1 0 0, limit effort=1 velocity=1
- added joint 0_to_26: type revolute, parent 0, child 26, origin xyz=0.09765164843013574 0.20035762048898975 0.11690241594468376 rpy=0.11396063374592824 3.320549569090366 4.698188204105016, axis 1 0 0, limit effort=1 velocity=1
