Commit message: hyper-parameter testing

File: URDF/0.urdf (robot description, URDF)
Before this commit: robot ted, 9 links, 8 joints
Links:
- removed link 15
- removed link 22
- removed link 23
- removed link 24
- removed link 26
- removed link 27
- removed link 28
- link 0: mass 0.6406075354898184 -> 0.7526891226514645; geometry collision cylinder length=0.054306300377287675 radius=0.5892146989850408; visual cylinder length=0.054306300377287675 radius=0.5892146989850408
- link 11: mass 0.21962730422956667 -> 0.9933860252397347; geometry collision cylinder length=0.09947828364326727 radius=0.06566944613952708; visual cylinder length=0.09947828364326727 radius=0.06566944613952708
Joints:
- removed joint 0_to_15
- removed joint 11_to_22
- removed joint 11_to_23
- removed joint 11_to_24
- removed joint 15_to_26
- removed joint 15_to_27
- removed joint 15_to_28
- joint 0_to_11: origin xyz=0.41173728907590745 0.7121282447210531 0.5824931766248451 rpy=9.772587138913252 6.135237077640203 4.673844728901479 -> xyz=0.5439193980779878 0.37444840678331615 0.7189470771365731 rpy=11.166033840113736 3.8542756614023634 6.040632625578819

File: URDF/1.urdf (robot description, URDF)
Before this commit: robot ted, 9 links, 8 joints
Links:
- removed link 23
- removed link 27
- removed link 28
- added link 13, mass 0.15636075680340045; collision cylinder length=0.09108404154715014 radius=0.572992621291648; visual cylinder length=0.09108404154715014 radius=0.572992621291648
- link 0: mass 0.6406075354898184 -> 0.7526891226514645; geometry collision cylinder length=0.054306300377287675 radius=0.5892146989850408; visual cylinder length=0.054306300377287675 radius=0.5892146989850408
- link 11: mass 0.21962730422956667 -> 0.15636075680340045; geometry collision cylinder length=0.09108404154715014 radius=0.572992621291648; visual cylinder length=0.09108404154715014 radius=0.572992621291648
- link 15: mass 0.21962730422956667 -> 0.15636075680340045; geometry collision cylinder length=0.09108404154715014 radius=0.572992621291648; visual cylinder length=0.09108404154715014 radius=0.572992621291648
- link 22: mass 0.41090573523269014 -> 0.9933860252397347; geometry collision cylinder length=0.09947828364326727 radius=0.06566944613952708; visual cylinder length=0.09947828364326727 radius=0.06566944613952708
- link 24: mass 0.41090573523269014 -> 0.9933860252397347; geometry collision cylinder length=0.09947828364326727 radius=0.06566944613952708; visual cylinder length=0.09947828364326727 radius=0.06566944613952708
- link 26: mass 0.41090573523269014 -> 0.9933860252397347; geometry collision cylinder length=0.09947828364326727 radius=0.06566944613952708; visual cylinder length=0.09947828364326727 radius=0.06566944613952708
Joints:
- removed joint 11_to_23
- removed joint 11_to_24
- removed joint 15_to_27
- removed joint 15_to_28
- added joint 0_to_13: type revolute, parent 0, child 13, origin xyz=0.8809305489802048 0.38411808954313476 0.20415605373873158 rpy=9.029776496640672 5.9951599234050486 1.8002804145308209, axis 1 0 0, limit effort=1 velocity=1
- added joint 13_to_24: type revolute, parent 13, child 24, origin xyz=0.5439193980779878 0.37444840678331615 0.7189470771365731 rpy=11.166033840113736 3.8542756614023634 6.040632625578819, axis 1 0 0, limit effort=1 velocity=1
- joint 0_to_11: origin xyz=0.41173728907590745 0.7121282447210531 0.5824931766248451 rpy=9.772587138913252 6.135237077640203 4.673844728901479 -> xyz=0.8809305489802048 0.38411808954313476 0.20415605373873158 rpy=6.019850997760448 5.9951599234050486 1.8002804145308209
- joint 0_to_15: origin xyz=0.41173728907590745 0.7121282447210531 0.5824931766248451 rpy=14.658880708369878 6.135237077640203 4.673844728901479 -> xyz=0.8809305489802048 0.38411808954313476 0.20415605373873158 rpy=12.039701995520897 5.9951599234050486 1.8002804145308209
- joint 11_to_22: origin xyz=0.953866148735442 0.6548537646260819 0.11013515940345642 rpy=2.102332137072244 1.5801231317912616 6.119977702978318 -> xyz=0.5439193980779878 0.37444840678331615 0.7189470771365731 rpy=11.166033840113736 3.8542756614023634 6.040632625578819
- joint 15_to_26: origin xyz=0.953866148735442 0.6548537646260819 0.11013515940345642 rpy=2.102332137072244 1.5801231317912616 6.119977702978318 -> xyz=0.5439193980779878 0.37444840678331615 0.7189470771365731 rpy=11.166033840113736 3.8542756614023634 6.040632625578819

File: URDF/10.urdf (robot description, URDF)
Before this commit: robot ted, 4 links, 3 joints
Links:
- added link 15, mass 0.6711498260449934; collision cylinder length=0.9652864167682644 radius=0.33823465779542594; visual cylinder length=0.9652864167682644 radius=0.33823465779542594
- added link 24, mass 0.7127951113808741; collision cylinder length=0.8348634392058716 radius=0.7027988697150571; visual cylinder length=0.8348634392058716 radius=0.7027988697150571
- added link 26, mass 0.7127951113808741; collision cylinder length=0.8348634392058716 radius=0.7027988697150571; visual cylinder length=0.8348634392058716 radius=0.7027988697150571
- added link 27, mass 0.7127951113808741; collision cylinder length=0.8348634392058716 radius=0.7027988697150571; visual cylinder length=0.8348634392058716 radius=0.7027988697150571
- added link 28, mass 0.7127951113808741; collision cylinder length=0.8348634392058716 radius=0.7027988697150571; visual cylinder length=0.8348634392058716 radius=0.7027988697150571
- link 0: mass 0.9576674501473837 -> 0.49963684145833387; geometry collision cylinder length=0.5062827424154303 radius=0.1290986605420673; visual cylinder length=0.5062827424154303 radius=0.1290986605420673
- link 11: mass 0.19260508477109606 -> 0.6711498260449934; geometry collision cylinder length=0.9652864167682644 radius=0.33823465779542594; visual cylinder length=0.9652864167682644 radius=0.33823465779542594
- link 22: mass 0.674776319926726 -> 0.7127951113808741; geometry collision cylinder length=0.8348634392058716 radius=0.7027988697150571; visual cylinder length=0.8348634392058716 radius=0.7027988697150571
- link 23: mass 0.674776319926726 -> 0.7127951113808741; geometry collision cylinder length=0.8348634392058716 radius=0.7027988697150571; visual cylinder length=0.8348634392058716 radius=0.7027988697150571
Joints:
- removed joint 0_to_22
- removed joint 0_to_23
- added joint 0_to_15: type revolute, parent 0, child 15, origin xyz=0.22051588196801397 0.9975477474468675 0.5965448079135393 rpy=1.555500434598927 5.232884694168904 3.18254411499066, axis 1 0 0, limit effort=1 velocity=1
- added joint 11_to_22: type revolute, parent 11, child 22, origin xyz=0.6134453270489266 0.9661692422955028 0.9346486078773736 rpy=4.478965226927246 0.10923977347080842 4.052870949044047, axis 1 0 0, limit effort=1 velocity=1
- added joint 11_to_23: type revolute, parent 11, child 23, origin xyz=0.6134453270489266 0.9661692422955028 0.9346486078773736 rpy=6.718447840390869 0.10923977347080842 4.052870949044047, axis 1 0 0, limit effort=1 velocity=1
- added joint 11_to_24: type revolute, parent 11, child 24, origin xyz=0.6134453270489266 0.9661692422955028 0.9346486078773736 rpy=8.957930453854493 0.10923977347080842 4.052870949044047, axis 1 0 0, limit effort=1 velocity=1
- added joint 15_to_26: type revolute, parent 15, child 26, origin xyz=0.6134453270489266 0.9661692422955028 0.9346486078773736 rpy=4.478965226927246 0.10923977347080842 4.052870949044047, axis 1 0 0, limit effort=1 velocity=1
- added joint 15_to_27: type revolute, parent 15, child 27, origin xyz=0.6134453270489266 0.9661692422955028 0.9346486078773736 rpy=6.718447840390869 0.10923977347080842 4.052870949044047, axis 1 0 0, limit effort=1 velocity=1
- added joint 15_to_28: type revolute, parent 15, child 28, origin xyz=0.6134453270489266 0.9661692422955028 0.9346486078773736 rpy=8.957930453854493 0.10923977347080842 4.052870949044047, axis 1 0 0, limit effort=1 velocity=1
- joint 0_to_11: origin xyz=0.0647123763930777 0.7159752044118834 0.7679146475609268 rpy=6.045929688295032 5.215080526362034 5.332975148900843 -> xyz=0.22051588196801397 0.9975477474468675 0.5965448079135393 rpy=1.037000289732618 5.232884694168904 3.18254411499066; type fixed -> revolute

File: URDF/11.urdf (robot description, URDF)
Before this commit: robot ted, 6 links, 5 joints
Links:
- removed link 12
- removed link 25
- added link 15, mass 0.6711498260449934; collision cylinder length=0.9652864167682644 radius=0.33823465779542594; visual cylinder length=0.9652864167682644 radius=0.33823465779542594
- added link 22, mass 0.7127951113808741; collision cylinder length=0.8348634392058716 radius=0.7027988697150571; visual cylinder length=0.8348634392058716 radius=0.7027988697150571
- added link 26, mass 0.7127951113808741; collision cylinder length=0.8348634392058716 radius=0.7027988697150571; visual cylinder length=0.8348634392058716 radius=0.7027988697150571
- added link 27, mass 0.7127951113808741; collision cylinder length=0.8348634392058716 radius=0.7027988697150571; visual cylinder length=0.8348634392058716 radius=0.7027988697150571
- added link 28, mass 0.7127951113808741; collision cylinder length=0.8348634392058716 radius=0.7027988697150571; visual cylinder length=0.8348634392058716 radius=0.7027988697150571
- link 0: mass 0.7457402298794583 -> 0.49963684145833387; geometry collision cylinder length=0.5062827424154303 radius=0.1290986605420673; visual cylinder length=0.5062827424154303 radius=0.1290986605420673
- link 11: mass 0.9059602521731824 -> 0.6711498260449934; geometry collision cylinder length=0.9652864167682644 radius=0.33823465779542594; visual cylinder length=0.9652864167682644 radius=0.33823465779542594
- link 23: mass 0.44736366272009565 -> 0.7127951113808741; geometry collision cylinder length=0.8348634392058716 radius=0.7027988697150571; visual cylinder length=0.8348634392058716 radius=0.7027988697150571
- link 24: mass 0.44736366272009565 -> 0.7127951113808741; geometry collision cylinder length=0.8348634392058716 radius=0.7027988697150571; visual cylinder length=0.8348634392058716 radius=0.7027988697150571
Joints:
- removed joint 0_to_12
- removed joint 0_to_23
- removed joint 0_to_24
- removed joint 0_to_25
- added joint 0_to_15: type revolute, parent 0, child 15, origin xyz=0.22051588196801397 0.9975477474468675 0.5965448079135393 rpy=1.555500434598927 5.232884694168904 3.18254411499066, axis 1 0 0, limit effort=1 velocity=1
- added joint 11_to_22: type revolute, parent 11, child 22, origin xyz=0.6134453270489266 0.9661692422955028 0.9346486078773736 rpy=4.478965226927246 0.10923977347080842 4.052870949044047, axis 1 0 0, limit effort=1 velocity=1
- added joint 11_to_23: type revolute, parent 11, child 23, origin xyz=0.6134453270489266 0.9661692422955028 0.9346486078773736 rpy=6.718447840390869 0.10923977347080842 4.052870949044047, axis 1 0 0, limit effort=1 velocity=1
- added joint 11_to_24: type revolute, parent 11, child 24, origin xyz=0.6134453270489266 0.9661692422955028 0.9346486078773736 rpy=8.957930453854493 0.10923977347080842 4.052870949044047, axis 1 0 0, limit effort=1 velocity=1
- added joint 15_to_26: type revolute, parent 15, child 26, origin xyz=0.6134453270489266 0.9661692422955028 0.9346486078773736 rpy=4.478965226927246 0.10923977347080842 4.052870949044047, axis 1 0 0, limit effort=1 velocity=1
- added joint 15_to_27: type revolute, parent 15, child 27, origin xyz=0.6134453270489266 0.9661692422955028 0.9346486078773736 rpy=6.718447840390869 0.10923977347080842 4.052870949044047, axis 1 0 0, limit effort=1 velocity=1
- added joint 15_to_28: type revolute, parent 15, child 28, origin xyz=0.6134453270489266 0.9661692422955028 0.9346486078773736 rpy=8.957930453854493 0.10923977347080842 4.052870949044047, axis 1 0 0, limit effort=1 velocity=1
- joint 0_to_11: origin xyz=0.3932748374880398 0.616263810309897 0.15444660257576093 rpy=9.63129901465597 0.5170502488772097 3.5920418865609864 -> xyz=0.22051588196801397 0.9975477474468675 0.5965448079135393 rpy=1.037000289732618 5.232884694168904 3.18254411499066

File: URDF/3.urdf (robot description, URDF)
Before this commit: robot ted, 9 links, 8 joints
Links:
- removed link 15
- removed link 22
- removed link 23
- removed link 24
- removed link 26
- removed link 27
- removed link 28
- added link 12, mass 0.15636075680340045; collision cylinder length=0.187087532994329 radius=0.572992621291648; visual cylinder length=0.187087532994329 radius=0.572992621291648
- added link 13, mass 0.15636075680340045; collision cylinder length=0.187087532994329 radius=0.572992621291648; visual cylinder length=0.187087532994329 radius=0.572992621291648
- link 0: mass 0.6406075354898184 -> 0.7526891226514645; geometry collision cylinder length=0.054306300377287675 radius=0.5892146989850408; visual cylinder length=0.054306300377287675 radius=0.5892146989850408
- link 11: mass 0.21962730422956667 -> 0.15636075680340045; geometry collision cylinder length=0.187087532994329 radius=0.572992621291648; visual cylinder length=0.187087532994329 radius=0.572992621291648
Joints:
- removed joint 0_to_15
- removed joint 11_to_22
- removed joint 11_to_23
- removed joint 11_to_24
- removed joint 15_to_26
- removed joint 15_to_27
- removed joint 15_to_28
- added joint 0_to_12: type revolute, parent 0, child 12, origin xyz=0.8809305489802048 0.38411808954313476 0.20415605373873158 rpy=9.029776496640672 5.9951599234050486 1.8002804145308209, axis 1 0 0, limit effort=1 velocity=1
- added joint 0_to_13: type revolute, parent 0, child 13, origin xyz=0.8809305489802048 0.38411808954313476 0.20415605373873158 rpy=12.039701995520897 5.9951599234050486 1.8002804145308209, axis 1 0 0, limit effort=1 velocity=1
- joint 0_to_11: origin xyz=0.41173728907590745 0.7121282447210531 0.5824931766248451 rpy=9.772587138913252 6.135237077640203 4.673844728901479 -> xyz=0.8809305489802048 0.38411808954313476 0.20415605373873158 rpy=6.019850997760448 5.9951599234050486 1.8002804145308209

File: URDF/4.urdf (robot description, URDF)
Before this commit: robot ted, 9 links, 8 joints
Links:
- removed link 15
- removed link 26
- removed link 27
- removed link 28
- added link 25, mass 0.08249661977674638; collision cylinder length=0.16063551896294537 radius=0.8597203587150178; visual cylinder length=0.16063551896294537 radius=0.8597203587150178
- link 0: mass 0.6406075354898184 -> 0.7526891226514645; geometry collision cylinder length=0.054306300377287675 radius=0.5892146989850408; visual cylinder length=0.054306300377287675 radius=0.5892146989850408
- link 11: mass 0.21962730422956667 -> 0.9933860252397347; geometry collision cylinder length=0.09947828364326727 radius=0.06566944613952708; visual cylinder length=0.09947828364326727 radius=0.06566944613952708
- link 22: mass 0.41090573523269014 -> 0.08249661977674638; geometry collision cylinder length=0.16063551896294537 radius=0.8597203587150178; visual cylinder length=0.16063551896294537 radius=0.8597203587150178
- link 23: mass 0.41090573523269014 -> 0.08249661977674638; geometry collision cylinder length=0.16063551896294537 radius=0.8597203587150178; visual cylinder length=0.16063551896294537 radius=0.8597203587150178
- link 24: mass 0.41090573523269014 -> 0.08249661977674638; geometry collision cylinder length=0.16063551896294537 radius=0.8597203587150178; visual cylinder length=0.16063551896294537 radius=0.8597203587150178
Joints:
- removed joint 0_to_15
- removed joint 11_to_22
- removed joint 11_to_23
- removed joint 11_to_24
- removed joint 15_to_26
- removed joint 15_to_27
- removed joint 15_to_28
- added joint 0_to_22: type revolute, parent 0, child 22, origin xyz=0.13446711138752465 0.33383683205248205 0.33318985105572585 rpy=17.794309710543555 4.053688992947098 4.732238250770481, axis 1 0 0, limit effort=1 velocity=1
- added joint 0_to_23: type revolute, parent 0, child 23, origin xyz=0.13446711138752465 0.33383683205248205 0.33318985105572585 rpy=23.72574628072474 4.053688992947098 4.732238250770481, axis 1 0 0, limit effort=1 velocity=1
- added joint 0_to_24: type revolute, parent 0, child 24, origin xyz=0.13446711138752465 0.33383683205248205 0.33318985105572585 rpy=29.657182850905922 4.053688992947098 4.732238250770481, axis 1 0 0, limit effort=1 velocity=1
- added joint 0_to_25: type revolute, parent 0, child 25, origin xyz=0.13446711138752465 0.33383683205248205 0.33318985105572585 rpy=35.58861942108711 4.053688992947098 4.732238250770481, axis 1 0 0, limit effort=1 velocity=1
- joint 0_to_11: origin xyz=0.41173728907590745 0.7121282447210531 0.5824931766248451 rpy=9.772587138913252 6.135237077640203 4.455457061760032 -> xyz=0.5439193980779878 0.37444840678331615 0.7189470771365731 rpy=11.166033840113736 3.8542756614023634 6.040632625578819

File: URDF/5.urdf (robot description, URDF)
Before this commit: robot ted, 9 links, 8 joints
Links:
- removed link 15
- removed link 22
- removed link 23
- removed link 26
- removed link 27
- removed link 28
- added link 12, mass 0.15636075680340045; collision cylinder length=0.187087532994329 radius=0.572992621291648; visual cylinder length=0.187087532994329 radius=0.572992621291648
- added link 13, mass 0.15636075680340045; collision cylinder length=0.187087532994329 radius=0.572992621291648; visual cylinder length=0.187087532994329 radius=0.572992621291648
- link 0: mass 0.6406075354898184 -> 0.7526891226514645; geometry collision cylinder length=0.054306300377287675 radius=0.5892146989850408; visual cylinder length=0.054306300377287675 radius=0.5892146989850408
- link 11: mass 0.21962730422956667 -> 0.15636075680340045; geometry collision cylinder length=0.187087532994329 radius=0.572992621291648; visual cylinder length=0.187087532994329 radius=0.572992621291648
- link 24: mass 0.41090573523269014 -> 0.08689524688268757; geometry collision cylinder length=0.8295505750604851 radius=0.41094524062472415; visual cylinder length=0.8295505750604851 radius=0.41094524062472415
Joints:
- removed joint 0_to_15
- removed joint 11_to_22
- removed joint 11_to_23
- removed joint 11_to_24
- removed joint 15_to_26
- removed joint 15_to_27
- removed joint 15_to_28
- added joint 0_to_12: type revolute, parent 0, child 12, origin xyz=0.8809305489802048 0.38411808954313476 0.20415605373873158 rpy=9.029776496640672 5.9951599234050486 1.8002804145308209, axis 1 0 0, limit effort=1 velocity=1
- added joint 0_to_13: type revolute, parent 0, child 13, origin xyz=0.8809305489802048 0.38411808954313476 0.20415605373873158 rpy=12.039701995520897 5.9951599234050486 1.8002804145308209, axis 1 0 0, limit effort=1 velocity=1
- added joint 0_to_24: type revolute, parent 0, child 24, origin xyz=0.2825394895248151 0.04871800868457221 0.6701991441175058 rpy=16.773013470252064 2.596152255905321 2.7060953779490973, axis 1 0 0, limit effort=1 velocity=1
- joint 0_to_11: origin xyz=0.41173728907590745 0.7121282447210531 0.5824931766248451 rpy=9.772587138913252 6.135237077640203 4.673844728901479 -> xyz=0.8809305489802048 0.38411808954313476 0.20415605373873158 rpy=6.019850997760448 5.9951599234050486 1.8002804145308209

File: URDF/6.urdf (robot description, URDF)
Before this commit: robot ted, 4 links, 3 joints
Links:
- removed link 12
- added link 15, mass 0.15636075680340045; collision cylinder length=0.187087532994329 radius=0.572992621291648; visual cylinder length=0.187087532994329 radius=0.572992621291648
- added link 22, mass 0.9933860252397347; collision cylinder length=0.09947828364326727 radius=0.06566944613952708; visual cylinder length=0.09947828364326727 radius=0.06566944613952708
- added link 24, mass 0.9933860252397347; collision cylinder length=0.09947828364326727 radius=0.06566944613952708; visual cylinder length=0.09947828364326727 radius=0.06566944613952708
- added link 26, mass 0.9933860252397347; collision cylinder length=0.09947828364326727 radius=0.06566944613952708; visual cylinder length=0.09947828364326727 radius=0.06566944613952708
- link 0: mass 0.6406075354898184 -> 0.7526891226514645; geometry collision cylinder length=0.054306300377287675 radius=0.5892146989850408; visual cylinder length=0.054306300377287675 radius=0.5892146989850408
- link 11: mass 0.41090573523269014 -> 0.15636075680340045; geometry collision cylinder length=0.187087532994329 radius=0.572992621291648; visual cylinder length=0.187087532994329 radius=0.572992621291648
- link 13: mass 0.41090573523269014 -> 0.15636075680340045; geometry collision cylinder length=0.187087532994329 radius=0.572992621291648; visual cylinder length=0.187087532994329 radius=0.572992621291648
Joints:
- removed joint 0_to_12
- added joint 0_to_15: type revolute, parent 0, child 15, origin xyz=0.8809305489802048 0.38411808954313476 0.20415605373873158 rpy=12.039701995520897 5.9951599234050486 1.8002804145308209, axis 1 0 0, limit effort=1 velocity=1
- added joint 11_to_22: type revolute, parent 11, child 22, origin xyz=0.5439193980779878 0.37444840678331615 0.7189470771365731 rpy=11.166033840113736 3.8542756614023634 6.040632625578819, axis 1 0 0, limit effort=1 velocity=1
- added joint 13_to_24: type revolute, parent 13, child 24, origin xyz=0.5439193980779878 0.37444840678331615 0.7189470771365731 rpy=11.166033840113736 3.8542756614023634 6.040632625578819, axis 1 0 0, limit effort=1 velocity=1
- added joint 15_to_26: type revolute, parent 15, child 26, origin xyz=0.5439193980779878 0.37444840678331615 0.7189470771365731 rpy=11.166033840113736 3.8542756614023634 6.040632625578819, axis 1 0 0, limit effort=1 velocity=1
- joint 0_to_11: origin xyz=0.953866148735442 0.6548537646260819 0.11013515940345642 rpy=2.102332137072244 1.5801231317912616 6.119977702978318 -> xyz=0.8809305489802048 0.38411808954313476 0.20415605373873158 rpy=6.019850997760448 5.9951599234050486 1.8002804145308209
- joint 0_to_13: origin xyz=0.953866148735442 0.6548537646260819 0.11013515940345642 rpy=4.204664274144488 1.5801231317912616 6.119977702978318 -> xyz=0.8809305489802048 0.38411808954313476 0.20415605373873158 rpy=9.029776496640672 5.9951599234050486 1.8002804145308209
