Commit message: hyper-parameter testing

File: URDF/7.urdf (robot description, URDF)
Before this commit: robot ted, 4 links, 3 joints
Links:
- removed link 12
- added link 15, mass 0.15636075680340045; collision cylinder length=0.187087532994329 radius=0.572992621291648; visual cylinder length=0.187087532994329 radius=0.572992621291648
- added link 22, mass 0.9933860252397347; collision cylinder length=0.09947828364326727 radius=0.06566944613952708; visual cylinder length=0.09947828364326727 radius=0.06566944613952708
- added link 24, mass 0.9933860252397347; collision cylinder length=0.09947828364326727 radius=0.06566944613952708; visual cylinder length=0.09947828364326727 radius=0.06566944613952708
- added link 26, mass 0.9933860252397347; collision cylinder length=0.09947828364326727 radius=0.06566944613952708; visual cylinder length=0.09947828364326727 radius=0.06566944613952708
- link 0: mass 0.21962730422956667 -> 0.7526891226514645; geometry collision cylinder length=0.054306300377287675 radius=0.5892146989850408; visual cylinder length=0.054306300377287675 radius=0.5892146989850408
- link 11: mass 0.41090573523269014 -> 0.15636075680340045; geometry collision cylinder length=0.187087532994329 radius=0.572992621291648; visual cylinder length=0.187087532994329 radius=0.572992621291648
- link 13: mass 0.41090573523269014 -> 0.15636075680340045; geometry collision cylinder length=0.187087532994329 radius=0.572992621291648; visual cylinder length=0.187087532994329 radius=0.572992621291648
Joints:
- removed joint 0_to_12
- added joint 0_to_15: type revolute, parent 0, child 15, origin xyz=0.8809305489802048 0.38411808954313476 0.20415605373873158 rpy=12.039701995520897 5.9951599234050486 1.8002804145308209, axis 1 0 0, limit effort=1 velocity=1
- added joint 11_to_22: type revolute, parent 11, child 22, origin xyz=0.5439193980779878 0.37444840678331615 0.7189470771365731 rpy=11.166033840113736 3.8542756614023634 6.040632625578819, axis 1 0 0, limit effort=1 velocity=1
- added joint 13_to_24: type revolute, parent 13, child 24, origin xyz=0.5439193980779878 0.37444840678331615 0.7189470771365731 rpy=11.166033840113736 3.8542756614023634 6.040632625578819, axis 1 0 0, limit effort=1 velocity=1
- added joint 15_to_26: type revolute, parent 15, child 26, origin xyz=0.5439193980779878 0.37444840678331615 0.7189470771365731 rpy=11.166033840113736 3.8542756614023634 6.040632625578819, axis 1 0 0, limit effort=1 velocity=1
- joint 0_to_11: origin xyz=0.953866148735442 0.6548537646260819 0.11013515940345642 rpy=2.102332137072244 1.5801231317912616 6.119977702978318 -> xyz=0.8809305489802048 0.38411808954313476 0.20415605373873158 rpy=6.019850997760448 5.9951599234050486 1.8002804145308209
- joint 0_to_13: origin xyz=0.953866148735442 0.6548537646260819 0.11013515940345642 rpy=4.204664274144488 1.5801231317912616 6.119977702978318 -> xyz=0.8809305489802048 0.38411808954313476 0.20415605373873158 rpy=9.029776496640672 5.9951599234050486 1.8002804145308209

File: URDF/8.urdf (robot description, URDF)
Before this commit: robot ted, 9 links, 8 joints
Links:
- removed link 15
- removed link 22
- removed link 23
- removed link 24
- removed link 26
- removed link 27
- removed link 28
- added link 12, mass 0.8028951187014396; collision cylinder length=0.6275206083791125 radius=0.6945119290396154; visual cylinder length=0.6275206083791125 radius=0.6945119290396154
- link 0: mass 0.6406075354898184 -> 0.7085418837834666; geometry collision cylinder length=0.6667815486691114 radius=0.7073958784216217; visual cylinder length=0.6667815486691114 radius=0.7073958784216217
- link 11: mass 0.21962730422956667 -> 0.8028951187014396; geometry collision cylinder length=0.6275206083791125 radius=0.6945119290396154; visual cylinder length=0.6275206083791125 radius=0.6945119290396154
Joints:
- removed joint 0_to_15
- removed joint 11_to_22
- removed joint 11_to_23
- removed joint 11_to_24
- removed joint 15_to_26
- removed joint 15_to_27
- removed joint 15_to_28
- added joint 0_to_12: type fixed, parent 0, child 12, origin xyz=0.5609096481571743 0.08103082987705568 0.35081288369713304 rpy=9.653144116812438 6.274901792805382 4.208692973810817, axis 1 0 0, limit effort=1 velocity=1
- joint 0_to_11: origin xyz=0.41173728907590745 0.7121282447210531 0.5824931766248451 rpy=9.772587138913252 6.135237077640203 4.673844728901479 -> xyz=0.5609096481571743 0.08103082987705568 0.35081288369713304 rpy=6.4354294112082915 6.274901792805382 4.208692973810817; type revolute -> fixed

File: URDF/9.urdf (robot description, URDF)
Before this commit: robot ted, 7 links, 6 joints
Links:
- removed link 23
- removed link 24
- removed link 25
- removed link 26
- added link 13, mass 0.840130841282373; collision cylinder length=0.4198534217419132 radius=0.5965588855925706; visual cylinder length=0.4198534217419132 radius=0.5965588855925706
- link 0: mass 0.6406075354898184 -> 0.7085418837834666; geometry collision cylinder length=0.6667815486691114 radius=0.7073958784216217; visual cylinder length=0.6667815486691114 radius=0.7073958784216217
- link 11: mass 0.21962730422956667 -> 0.840130841282373; geometry collision cylinder length=0.4198534217419132 radius=0.5965588855925706; visual cylinder length=0.4198534217419132 radius=0.5965588855925706
- link 12: mass 0.21962730422956667 -> 0.840130841282373; geometry collision cylinder length=0.4198534217419132 radius=0.5965588855925706; visual cylinder length=0.4198534217419132 radius=0.5965588855925706
Joints:
- removed joint 0_to_23
- removed joint 0_to_24
- removed joint 0_to_25
- removed joint 0_to_26
- added joint 0_to_13: type fixed, parent 0, child 13, origin xyz=0.8752961393334611 0.743563824546788 0.482262135334239 rpy=14.956126191911387 1.3152879553850032 5.016106402428998, axis 1 0 0, limit effort=1 velocity=1
- joint 0_to_11: origin xyz=0.41173728907590745 0.7121282447210531 0.5824931766248451 rpy=9.772587138913252 6.135237077640203 4.673844728901479 -> xyz=0.8752961393334611 0.743563824546788 0.482262135334239 rpy=7.478063095955694 1.3152879553850032 5.016106402428998; type revolute -> fixed
- joint 0_to_12: origin xyz=0.41173728907590745 0.7121282447210531 0.5824931766248451 rpy=14.658880708369878 6.135237077640203 4.673844728901479 -> xyz=0.8752961393334611 0.743563824546788 0.482262135334239 rpy=11.21709464393354 1.3152879553850032 5.016106402428998; type revolute -> fixed
